Commit message: some issues still but things are moving in rviz

File: urdf/human_scaled.urdf (robot description, URDF)
Before this commit: robot human_scaled, 80 links, 79 joints
Links:
- link left_foot: geometry visual mesh filename=package://rtcosmik_ros/meshes/foot_mesh.STL scale=0.006700 0.006700 0.006700
- link left_hand: geometry visual mesh filename=package://rtcosmik_ros/meshes/hand_mesh.STL scale=0.006100 0.006100 0.006100
- link left_lowerarm: geometry visual mesh filename=package://rtcosmik_ros/meshes/elbow_mesh.STL scale=0.005500 0.005500 0.005500; visual mesh filename=package://rtcosmik_ros/meshes/lowerarm_mesh.STL scale=0.006400 0.006400 0.006400
- link left_lowerleg: geometry visual mesh filename=package://rtcosmik_ros/meshes/knee_mesh.STL scale=0.005700 0.005700 0.005700; visual mesh filename=package://rtcosmik_ros/meshes/lowerleg_mesh.STL scale=0.006300 0.006600 0.007100
- link left_upperarm: geometry visual mesh filename=package://rtcosmik_ros/meshes/shoulder_mesh.STL scale=0.003900 0.003900 0.003900; visual mesh filename=package://rtcosmik_ros/meshes/upperarm_mesh.STL scale=0.006300 0.006000 0.007000
- link left_upperleg: geometry visual mesh filename=package://rtcosmik_ros/meshes/upperleg_mesh.STL scale=0.006200 0.006400 0.007000
- link middle_abdomen: geometry visual mesh filename=package://rtcosmik_ros/meshes/abdomen_mesh.STL scale=0.007500 0.007500 0.007500
- link middle_head: geometry visual mesh filename=package://rtcosmik_ros/meshes/head_mesh.STL scale=0.005600 0.005600 0.005600; visual mesh filename=package://rtcosmik_ros/meshes/neck_mesh.STL scale=0.005000 0.005000 0.005000
- link middle_pelvis: geometry visual mesh filename=package://rtcosmik_ros/meshes/pelvis_mesh.STL scale=0.006400 0.005800 0.005800
- link middle_thorax: geometry visual mesh filename=package://rtcosmik_ros/meshes/torso_mesh.STL scale=0.007200 0.007200 0.007200
- link right_foot: geometry visual mesh filename=package://rtcosmik_ros/meshes/foot_mesh.STL scale=0.006700 0.006700 0.006700
- link right_hand: geometry visual mesh filename=package://rtcosmik_ros/meshes/hand_mesh.STL scale=0.006100 0.006100 0.006100
- link right_lowerarm: geometry visual mesh filename=package://rtcosmik_ros/meshes/elbow_mesh.STL scale=0.005500 0.005500 0.005500; visual mesh filename=package://rtcosmik_ros/meshes/lowerarm_mesh.STL scale=0.006400 0.006400 0.006400
- link right_lowerleg: geometry visual mesh filename=package://rtcosmik_ros/meshes/knee_mesh.STL scale=0.005700 0.005700 0.005700; visual mesh filename=package://rtcosmik_ros/meshes/lowerleg_mesh.STL scale=0.006300 0.006600 0.007100
- link right_upperarm: geometry visual mesh filename=package://rtcosmik_ros/meshes/shoulder_mesh.STL scale=0.003900 0.003900 0.003900; visual mesh filename=package://rtcosmik_ros/meshes/upperarm_mesh.STL scale=0.006300 0.006000 0.007000
- link right_upperleg: geometry visual mesh filename=package://rtcosmik_ros/meshes/upperleg_mesh.STL scale=0.006200 0.006400 0.007000
Joints:
- joint joint_C7: origin xyz=-0.117128 0.199709 -0.032455 rpy=0.000000 -0.000000 0.000000 -> xyz=-0.084941 0.064655 -0.007302 rpy=0.000000 -0.000000 0.000000
- joint joint_Head: origin xyz=-0.175489 0.264136 -0.008885 rpy=0.000000 -0.000000 0.000000 -> xyz=-0.126054 0.215579 -0.003306 rpy=0.000000 -0.000000 0.000000
- joint joint_L5MHD: origin xyz=0.135335 0.026282 0.049689 rpy=0.000000 -0.000000 0.000000 -> xyz=0.134404 -0.000924 0.030323 rpy=0.000000 -0.000000 0.000000
- joint joint_LANK: origin xyz=0.027298 -0.199245 0.075142 rpy=0.000000 -0.000000 0.000000 -> xyz=0.030276 -0.222941 0.070394 rpy=0.000000 -0.000000 0.000000
- joint joint_LASI: origin xyz=0.101089 0.148047 -0.053473 rpy=0.000000 -0.000000 0.000000 -> xyz=0.105616 -0.035391 -0.078379 rpy=0.000000 -0.000000 0.000000
- joint joint_LELB: origin xyz=-0.012190 -0.294863 0.073364 rpy=0.000000 -0.000000 0.000000 -> xyz=0.014243 -0.171973 -0.021030 rpy=0.000000 -0.000000 0.000000
- joint joint_LEar: origin xyz=-0.179292 0.204914 0.073094 rpy=0.000000 -0.000000 0.000000 -> xyz=-0.055802 0.152346 0.026541 rpy=0.000000 -0.000000 0.000000
- joint joint_LEye: origin xyz=-0.138266 0.196150 0.011371 rpy=0.000000 -0.000000 0.000000 -> xyz=-0.110921 0.146401 -0.017645 rpy=0.000000 -0.000000 0.000000
- joint joint_LHEE: origin xyz=-0.172566 0.001149 0.090394 rpy=0.000000 -0.000000 0.000000 -> xyz=-0.155587 -0.017775 0.077763 rpy=0.000000 -0.000000 0.000000
- joint joint_LKNE: origin xyz=0.016330 -0.356700 -0.004916 rpy=0.000000 -0.000000 0.000000 -> xyz=0.039518 -0.370630 0.067066 rpy=0.000000 -0.000000 0.000000
- joint joint_LMANK: origin xyz=-0.001947 -0.228416 0.060052 rpy=0.000000 -0.000000 0.000000 -> xyz=-0.000321 -0.240511 0.050212 rpy=0.000000 -0.000000 0.000000
- joint joint_LMELB: origin xyz=-0.056616 -0.299666 0.045797 rpy=0.000000 -0.000000 0.000000 -> xyz=0.001025 -0.166220 0.025358 rpy=0.000000 -0.000000 0.000000
- joint joint_LMID: origin xyz=-0.004222 -0.170619 -0.000116 rpy=0.000000 -0.000000 0.000000 -> xyz=-0.001051 -0.082816 -0.001666 rpy=0.000000 -0.000000 0.000000
- joint joint_LMKNE: origin xyz=-0.050660 -0.316323 -0.016927 rpy=0.000000 -0.000000 0.000000 -> xyz=-0.031816 -0.357857 0.048251 rpy=0.000000 -0.000000 0.000000
- joint joint_LMWRI: origin xyz=0.001407 -0.265498 0.022654 rpy=0.000000 -0.000000 0.000000 -> xyz=0.000139 -0.160634 0.003574 rpy=0.000000 -0.000000 0.000000
- joint joint_LPIN: origin xyz=-0.013580 -0.177269 0.027270 rpy=0.000000 -0.000000 0.000000 -> xyz=-0.000342 -0.086310 0.017972 rpy=0.000000 -0.000000 0.000000
- joint joint_LPSI: origin xyz=0.023554 0.077151 -0.017341 rpy=0.000000 -0.000000 0.000000 -> xyz=0.055791 -0.032425 0.006519 rpy=0.000000 -0.000000 0.000000
- joint joint_LSHO: origin xyz=-0.109112 -0.093183 0.253402 rpy=0.000000 -0.000000 0.000000 -> xyz=-0.057218 0.003328 0.094644 rpy=0.000000 -0.000000 0.000000
- joint joint_LTHU: origin xyz=-0.006509 -0.162291 -0.033311 rpy=0.000000 -0.000000 0.000000 -> xyz=-0.010119 -0.079524 -0.014773 rpy=0.000000 -0.000000 0.000000
- joint joint_LTOE: origin xyz=0.153426 -0.039447 0.052868 rpy=0.000000 -0.000000 0.000000 -> xyz=0.146787 -0.060555 0.016339 rpy=0.000000 -0.000000 0.000000
- joint joint_LWRI: origin xyz=0.002056 -0.257366 -0.002101 rpy=0.000000 -0.000000 0.000000 -> xyz=-0.005977 -0.157624 -0.008569 rpy=0.000000 -0.000000 0.000000
- joint joint_Nose: origin xyz=-0.143891 0.159003 -0.006287 rpy=0.000000 -0.000000 0.000000 -> xyz=-0.132215 0.113423 -0.005239 rpy=0.000000 -0.000000 0.000000
- joint joint_R5MHD: origin xyz=0.065121 0.037075 -0.007662 rpy=0.000000 -0.000000 0.000000 -> xyz=0.079074 0.012125 -0.011798 rpy=0.000000 -0.000000 0.000000
- joint joint_RANK: origin xyz=0.040331 -0.200559 0.017267 rpy=0.000000 -0.000000 0.000000 -> xyz=0.023027 -0.221148 0.014618 rpy=0.000000 -0.000000 0.000000
- joint joint_RASI: origin xyz=-0.025819 0.065977 -0.148658 rpy=0.000000 -0.000000 0.000000 -> xyz=-0.026713 -0.127009 -0.026761 rpy=0.000000 -0.000000 0.000000
- joint joint_RELB: origin xyz=-0.049061 -0.290829 -0.040308 rpy=0.000000 -0.000000 0.000000 -> xyz=-0.037312 -0.203387 0.012616 rpy=0.000000 -0.000000 0.000000
- joint joint_REar: origin xyz=-0.239153 0.168132 -0.003877 rpy=0.000000 -0.000000 0.000000 -> xyz=-0.143667 0.136693 0.074293 rpy=0.000000 -0.000000 0.000000
- joint joint_REye: origin xyz=-0.171318 0.181389 -0.023664 rpy=0.000000 -0.000000 0.000000 -> xyz=-0.150083 0.140111 0.010372 rpy=0.000000 -0.000000 0.000000
- joint joint_RHEE: origin xyz=-0.087564 0.043859 -0.209942 rpy=0.000000 -0.000000 0.000000 -> xyz=-0.095167 0.087533 -0.171143 rpy=0.000000 -0.000000 0.000000
- joint joint_RKNE: origin xyz=-0.073559 -0.359489 -0.002676 rpy=0.000000 -0.000000 0.000000 -> xyz=-0.082840 -0.330213 0.006352 rpy=0.000000 -0.000000 0.000000
- joint joint_RMANK: origin xyz=0.059236 -0.224417 -0.029898 rpy=0.000000 -0.000000 0.000000 -> xyz=0.057018 -0.232624 -0.017887 rpy=0.000000 -0.000000 0.000000
- joint joint_RMELB: origin xyz=-0.055154 -0.292699 0.007025 rpy=0.000000 -0.000000 0.000000 -> xyz=0.002674 -0.189291 0.026332 rpy=0.000000 -0.000000 0.000000
- joint joint_RMID: origin xyz=-0.004414 -0.168975 0.000558 rpy=0.000000 -0.000000 0.000000 -> xyz=-0.000994 -0.095388 0.000260 rpy=0.000000 -0.000000 0.000000
- joint joint_RMKNE: origin xyz=-0.032428 -0.366749 -0.079316 rpy=0.000000 -0.000000 0.000000 -> xyz=-0.020001 -0.351132 -0.045337 rpy=0.000000 -0.000000 0.000000
- joint joint_RMWRI: origin xyz=0.012764 -0.258366 -0.015537 rpy=0.000000 -0.000000 0.000000 -> xyz=0.005736 -0.177723 -0.000964 rpy=0.000000 -0.000000 0.000000
- joint joint_RPIN: origin xyz=-0.009225 -0.173833 -0.017551 rpy=0.000000 -0.000000 0.000000 -> xyz=-0.009705 -0.097698 -0.011634 rpy=0.000000 -0.000000 0.000000
- joint joint_RPSI: origin xyz=-0.027334 0.045470 -0.058243 rpy=0.000000 -0.000000 0.000000 -> xyz=0.001443 -0.070926 0.027163 rpy=0.000000 -0.000000 0.000000
- joint joint_RSHO: origin xyz=-0.080950 -0.072080 -0.271258 rpy=0.000000 -0.000000 0.000000 -> xyz=-0.070143 -0.009368 -0.182813 rpy=0.000000 -0.000000 0.000000
- joint joint_RTHU: origin xyz=-0.006709 -0.153663 0.016087 rpy=0.000000 -0.000000 0.000000 -> xyz=-0.001947 -0.085940 0.015163 rpy=0.000000 -0.000000 0.000000
- joint joint_RTOE: origin xyz=0.139544 -0.001610 -0.067527 rpy=0.000000 -0.000000 0.000000 -> xyz=0.134833 -0.012615 -0.082973 rpy=0.000000 -0.000000 0.000000
- joint joint_RWRI: origin xyz=0.012384 -0.252118 -0.001697 rpy=0.000000 -0.000000 0.000000 -> xyz=0.006651 -0.174416 0.011408 rpy=0.000000 -0.000000 0.000000
- joint joint_T11: origin xyz=0.024098 0.136632 -0.099270 rpy=0.000000 -0.000000 0.000000 -> xyz=0.006878 0.077403 0.013371 rpy=0.000000 -0.000000 0.000000
- joint joint_T6: origin xyz=-0.042073 0.134267 -0.032728 rpy=0.000000 -0.000000 0.000000 -> xyz=-0.013201 0.005432 0.015524 rpy=0.000000 -0.000000 0.000000
- joint left_ankle_Z: origin xyz=0.000000 -0.262180 0.000000 rpy=0.000000 -0.000000 0.000000 -> xyz=0.000000 -0.253410 0.000000 rpy=0.000000 -0.000000 0.000000
- joint left_clavicle_joint_X: origin xyz=0.000000 0.453718 0.000000 rpy=0.000000 -0.000000 0.000000 -> xyz=0.000000 0.162423 0.000000 rpy=0.000000 -0.000000 0.000000
- joint left_elbow_Z: origin xyz=0.000000 -0.175917 0.000000 rpy=0.000000 -0.000000 0.000000 -> xyz=0.000000 -0.170387 0.000000 rpy=0.000000 -0.000000 0.000000
- joint left_hip_Z: origin xyz=-0.009838 -0.066212 -0.064348 rpy=0.000000 -0.000000 0.000000 -> xyz=-0.012606 -0.062441 -0.061119 rpy=0.000000 -0.000000 0.000000
- joint left_knee_Z: origin xyz=0.000000 -0.398760 0.000000 rpy=0.000000 -0.000000 0.000000 -> xyz=0.000000 -0.385097 0.000000 rpy=0.000000 -0.000000 0.000000
- joint left_shoulder_Z: origin xyz=-0.018692 -0.034767 0.107550 rpy=0.000000 -0.000000 0.000000 -> xyz=-0.022196 -0.034218 0.104014 rpy=0.000000 -0.000000 0.000000
- joint left_wrist_Z: origin xyz=0.000000 -0.165186 0.000000 rpy=0.000000 -0.000000 0.000000 -> xyz=0.000000 -0.160850 0.000000 rpy=0.000000 -0.000000 0.000000
- joint middle_cervical_Z: origin xyz=0.000000 0.492561 0.000000 rpy=0.000000 -0.000000 0.000000 -> xyz=0.000000 0.217251 0.000000 rpy=0.000000 -0.000000 0.000000
- joint middle_thoracic_Z: origin xyz=0.000000 0.142922 0.000000 rpy=0.000000 -0.000000 0.000000 -> xyz=0.000000 0.144338 0.000000 rpy=0.000000 -0.000000 0.000000
- joint right_ankle_Z: origin xyz=0.000000 -0.258352 0.000000 rpy=0.000000 -0.000000 0.000000 -> xyz=0.000000 -0.253254 0.000000 rpy=0.000000 -0.000000 0.000000
- joint right_clavicle_joint_X: origin xyz=0.000000 0.453718 0.000000 rpy=0.000000 -0.000000 0.000000 -> xyz=0.000000 0.162423 0.000000 rpy=0.000000 -0.000000 0.000000
- joint right_elbow_Z: origin xyz=0.000000 -0.173497 0.000000 rpy=0.000000 -0.000000 0.000000 -> xyz=0.000000 -0.168042 0.000000 rpy=0.000000 -0.000000 0.000000
- joint right_hip_Z: origin xyz=-0.009838 -0.065959 0.064608 rpy=0.000000 -0.000000 0.000000 -> xyz=-0.012606 -0.062638 0.060917 rpy=0.000000 -0.000000 0.000000
- joint right_knee_Z: origin xyz=0.000000 -0.387276 0.000000 rpy=0.000000 -0.000000 0.000000 -> xyz=0.000000 -0.373432 0.000000 rpy=0.000000 -0.000000 0.000000
- joint right_shoulder_Z: origin xyz=0.018692 -0.039481 -0.107550 rpy=0.000000 -0.000000 0.000000 -> xyz=0.022196 -0.038116 -0.104014 rpy=0.000000 -0.000000 0.000000
- joint right_wrist_Z: origin xyz=0.000000 -0.162468 0.000000 rpy=0.000000 -0.000000 0.000000 -> xyz=0.000000 -0.156657 0.000000 rpy=0.000000 -0.000000 0.000000

Commit message: timestamped messages

File: urdf/human_scaled.urdf (robot description, URDF)
Before this commit: robot human_scaled, 80 links, 79 joints
Joints:
- joint joint_C7: origin xyz=-0.084941 0.064655 -0.007302 rpy=0.000000 -0.000000 0.000000 -> xyz=-0.088296 0.568608 0.022895 rpy=0.000000 -0.000000 0.000000
- joint joint_Head: origin xyz=-0.126054 0.215579 -0.003306 rpy=0.000000 -0.000000 0.000000 -> xyz=-0.063170 0.190906 -0.017908 rpy=0.000000 -0.000000 0.000000
- joint joint_L5MHD: origin xyz=0.134404 -0.000924 0.030323 rpy=0.000000 -0.000000 0.000000 -> xyz=0.149075 -0.028134 0.077726 rpy=0.000000 -0.000000 0.000000
- joint joint_LANK: origin xyz=0.030276 -0.222941 0.070394 rpy=0.000000 -0.000000 0.000000 -> xyz=0.020762 -0.408001 -0.021350 rpy=0.000000 -0.000000 0.000000
- joint joint_LASI: origin xyz=0.105616 -0.035391 -0.078379 rpy=0.000000 -0.000000 0.000000 -> xyz=-0.032298 0.225521 0.042993 rpy=0.000000 -0.000000 0.000000
- joint joint_LELB: origin xyz=0.014243 -0.171973 -0.021030 rpy=0.000000 -0.000000 0.000000 -> xyz=0.005704 -0.316023 -0.013916 rpy=0.000000 -0.000000 0.000000
- joint joint_LEar: origin xyz=-0.055802 0.152346 0.026541 rpy=0.000000 -0.000000 0.000000 -> xyz=-0.014424 0.067292 -0.069737 rpy=0.000000 -0.000000 0.000000
- joint joint_LEye: origin xyz=-0.110921 0.146401 -0.017645 rpy=0.000000 -0.000000 0.000000 -> xyz=0.073003 0.141644 -0.056717 rpy=0.000000 -0.000000 0.000000
- joint joint_LHEE: origin xyz=-0.155587 -0.017775 0.077763 rpy=0.000000 -0.000000 0.000000 -> xyz=-0.241040 -0.036928 0.119340 rpy=0.000000 -0.000000 0.000000
- joint joint_LKNE: origin xyz=0.039518 -0.370630 0.067066 rpy=0.000000 -0.000000 0.000000 -> xyz=0.010368 -0.359988 -0.049023 rpy=0.000000 -0.000000 0.000000
- joint joint_LMANK: origin xyz=-0.000321 -0.240511 0.050212 rpy=0.000000 -0.000000 0.000000 -> xyz=-0.023774 -0.406030 0.031546 rpy=0.000000 -0.000000 0.000000
- joint joint_LMELB: origin xyz=0.001025 -0.166220 0.025358 rpy=0.000000 -0.000000 0.000000 -> xyz=-0.033072 -0.327266 0.067426 rpy=0.000000 -0.000000 0.000000
- joint joint_LMID: origin xyz=-0.001051 -0.082816 -0.001666 rpy=0.000000 -0.000000 0.000000 -> xyz=0.000859 -0.151239 -0.000883 rpy=0.000000 -0.000000 0.000000
- joint joint_LMKNE: origin xyz=-0.031816 -0.357857 0.048251 rpy=0.000000 -0.000000 0.000000 -> xyz=-0.063080 -0.290571 0.011084 rpy=0.000000 -0.000000 0.000000
- joint joint_LMWRI: origin xyz=0.000139 -0.160634 0.003574 rpy=0.000000 -0.000000 0.000000 -> xyz=-0.013293 -0.286383 0.026804 rpy=0.000000 -0.000000 0.000000
- joint joint_LPIN: origin xyz=-0.000342 -0.086310 0.017972 rpy=0.000000 -0.000000 0.000000 -> xyz=0.013130 -0.166097 0.060680 rpy=0.000000 -0.000000 0.000000
- joint joint_LPSI: origin xyz=0.055791 -0.032425 0.006519 rpy=0.000000 -0.000000 0.000000 -> xyz=-0.184575 0.087863 0.019108 rpy=0.000000 -0.000000 0.000000
- joint joint_LSHO: origin xyz=-0.057218 0.003328 0.094644 rpy=0.000000 -0.000000 0.000000 -> xyz=0.006880 -0.041848 -0.155752 rpy=0.000000 -0.000000 0.000000
- joint joint_LTHU: origin xyz=-0.010119 -0.079524 -0.014773 rpy=0.000000 -0.000000 0.000000 -> xyz=0.001630 -0.133798 -0.067962 rpy=0.000000 -0.000000 0.000000
- joint joint_LTOE: origin xyz=0.146787 -0.060555 0.016339 rpy=0.000000 -0.000000 0.000000 -> xyz=0.134847 -0.045692 0.155654 rpy=0.000000 -0.000000 0.000000
- joint joint_LWRI: origin xyz=-0.005977 -0.157624 -0.008569 rpy=0.000000 -0.000000 0.000000 -> xyz=-0.012270 -0.278828 -0.031263 rpy=0.000000 -0.000000 0.000000
- joint joint_Nose: origin xyz=-0.132215 0.113423 -0.005239 rpy=0.000000 -0.000000 0.000000 -> xyz=0.125446 0.128348 -0.023599 rpy=0.000000 -0.000000 0.000000
- joint joint_R5MHD: origin xyz=0.079074 0.012125 -0.011798 rpy=0.000000 -0.000000 0.000000 -> xyz=0.157476 -0.035910 -0.043982 rpy=0.000000 -0.000000 0.000000
- joint joint_RANK: origin xyz=0.023027 -0.221148 0.014618 rpy=0.000000 -0.000000 0.000000 -> xyz=0.017420 -0.398158 0.034951 rpy=0.000000 -0.000000 0.000000
- joint joint_RASI: origin xyz=-0.026713 -0.127009 -0.026761 rpy=0.000000 -0.000000 0.000000 -> xyz=0.023423 0.026316 0.173711 rpy=0.000000 -0.000000 0.000000
- joint joint_RELB: origin xyz=-0.037312 -0.203387 0.012616 rpy=0.000000 -0.000000 0.000000 -> xyz=-0.014785 -0.320281 0.032681 rpy=0.000000 -0.000000 0.000000
- joint joint_REar: origin xyz=-0.143667 0.136693 0.074293 rpy=0.000000 -0.000000 0.000000 -> xyz=-0.004108 0.096011 0.084225 rpy=0.000000 -0.000000 0.000000
- joint joint_REye: origin xyz=-0.150083 0.140111 0.010372 rpy=0.000000 -0.000000 0.000000 -> xyz=0.075094 0.151108 0.013567 rpy=0.000000 -0.000000 0.000000
- joint joint_RHEE: origin xyz=-0.095167 0.087533 -0.171143 rpy=0.000000 -0.000000 0.000000 -> xyz=-0.254177 -0.034181 -0.110385 rpy=0.000000 -0.000000 0.000000
- joint joint_RKNE: origin xyz=-0.082840 -0.330213 0.006352 rpy=0.000000 -0.000000 0.000000 -> xyz=0.010147 -0.379736 0.016104 rpy=0.000000 -0.000000 0.000000
- joint joint_RMANK: origin xyz=0.057018 -0.232624 -0.017887 rpy=0.000000 -0.000000 0.000000 -> xyz=-0.009697 -0.403449 -0.031248 rpy=0.000000 -0.000000 0.000000
- joint joint_RMELB: origin xyz=0.002674 -0.189291 0.026332 rpy=0.000000 -0.000000 0.000000 -> xyz=-0.029558 -0.327197 -0.052072 rpy=0.000000 -0.000000 0.000000
- joint joint_RMID: origin xyz=-0.000994 -0.095388 0.000260 rpy=0.000000 -0.000000 0.000000 -> xyz=0.001853 -0.176359 0.000040 rpy=0.000000 -0.000000 0.000000
- joint joint_RMKNE: origin xyz=-0.020001 -0.351132 -0.045337 rpy=0.000000 -0.000000 0.000000 -> xyz=-0.074963 -0.393659 -0.068235 rpy=0.000000 -0.000000 0.000000
- joint joint_RMWRI: origin xyz=0.005736 -0.177723 -0.000964 rpy=0.000000 -0.000000 0.000000 -> xyz=-0.010818 -0.311185 -0.018371 rpy=0.000000 -0.000000 0.000000
- joint joint_RPIN: origin xyz=-0.009705 -0.097698 -0.011634 rpy=0.000000 -0.000000 0.000000 -> xyz=0.009811 -0.190681 -0.040969 rpy=0.000000 -0.000000 0.000000
- joint joint_RPSI: origin xyz=0.001443 -0.070926 0.027163 rpy=0.000000 -0.000000 0.000000 -> xyz=-0.151028 -0.003926 0.083364 rpy=0.000000 -0.000000 0.000000
- joint joint_RSHO: origin xyz=-0.070143 -0.009368 -0.182813 rpy=0.000000 -0.000000 0.000000 -> xyz=-0.038804 -0.004832 0.216822 rpy=0.000000 -0.000000 0.000000
- joint joint_RTHU: origin xyz=-0.001947 -0.085940 0.015163 rpy=0.000000 -0.000000 0.000000 -> xyz=0.006359 -0.148331 0.039116 rpy=0.000000 -0.000000 0.000000
- joint joint_RTOE: origin xyz=0.134833 -0.012615 -0.082973 rpy=0.000000 -0.000000 0.000000 -> xyz=0.169712 -0.037041 -0.150108 rpy=0.000000 -0.000000 0.000000
- joint joint_RWRI: origin xyz=0.006651 -0.174416 0.011408 rpy=0.000000 -0.000000 0.000000 -> xyz=-0.010523 -0.299224 0.016849 rpy=0.000000 -0.000000 0.000000
- joint joint_T11: origin xyz=0.006878 0.077403 0.013371 rpy=0.000000 -0.000000 0.000000 -> xyz=-0.168156 0.274745 0.230525 rpy=0.000000 -0.000000 0.000000
- joint joint_T6: origin xyz=-0.013201 0.005432 0.015524 rpy=0.000000 -0.000000 0.000000 -> xyz=-0.126739 0.420060 0.028283 rpy=0.000000 -0.000000 0.000000
- joint left_ankle_Z: origin xyz=0.000000 -0.253410 0.000000 rpy=0.000000 -0.000000 0.000000 -> xyz=0.000000 -0.438307 0.000000 rpy=0.000000 -0.000000 0.000000
- joint left_clavicle_joint_X: origin xyz=0.000000 0.162423 0.000000 rpy=0.000000 -0.000000 0.000000 -> xyz=0.000000 0.618421 0.000000 rpy=0.000000 -0.000000 0.000000
- joint left_elbow_Z: origin xyz=0.000000 -0.170387 0.000000 rpy=0.000000 -0.000000 0.000000 -> xyz=0.000000 -0.288015 0.000000 rpy=0.000000 -0.000000 0.000000
- joint left_hip_Z: origin xyz=-0.012606 -0.062441 -0.061119 rpy=0.000000 -0.000000 0.000000 -> xyz=0.022765 -0.090673 -0.088195 rpy=0.000000 -0.000000 0.000000
- joint left_knee_Z: origin xyz=0.000000 -0.385097 0.000000 rpy=0.000000 -0.000000 0.000000 -> xyz=0.000000 -0.395648 0.000000 rpy=0.000000 -0.000000 0.000000
- joint left_shoulder_Z: origin xyz=-0.022196 -0.034218 0.104014 rpy=0.000000 -0.000000 0.000000 -> xyz=-0.001037 -0.056159 -0.168760 rpy=0.000000 -0.000000 0.000000
- joint left_wrist_Z: origin xyz=0.000000 -0.160850 0.000000 rpy=0.000000 -0.000000 0.000000 -> xyz=0.000000 -0.256851 0.000000 rpy=0.000000 -0.000000 0.000000
- joint middle_cervical_Z: origin xyz=0.000000 0.217251 0.000000 rpy=0.000000 -0.000000 0.000000 -> xyz=0.000000 0.642803 0.000000 rpy=0.000000 -0.000000 0.000000
- joint middle_thoracic_Z: origin xyz=0.000000 0.144338 0.000000 rpy=0.000000 -0.000000 0.000000 -> xyz=0.000000 0.146114 0.000000 rpy=0.000000 -0.000000 0.000000
- joint right_ankle_Z: origin xyz=0.000000 -0.253254 0.000000 rpy=0.000000 -0.000000 0.000000 -> xyz=0.000000 -0.418762 0.000000 rpy=0.000000 -0.000000 0.000000
- joint right_clavicle_joint_X: origin xyz=0.000000 0.162423 0.000000 rpy=0.000000 -0.000000 0.000000 -> xyz=0.000000 0.618421 0.000000 rpy=0.000000 -0.000000 0.000000
- joint right_elbow_Z: origin xyz=0.000000 -0.168042 0.000000 rpy=0.000000 -0.000000 0.000000 -> xyz=0.000000 -0.274470 0.000000 rpy=0.000000 -0.000000 0.000000
- joint right_hip_Z: origin xyz=-0.012606 -0.062638 0.060917 rpy=0.000000 -0.000000 0.000000 -> xyz=0.022765 -0.090400 0.088474 rpy=0.000000 -0.000000 0.000000
- joint right_knee_Z: origin xyz=0.000000 -0.373432 0.000000 rpy=0.000000 -0.000000 0.000000 -> xyz=0.000000 -0.402147 0.000000 rpy=0.000000 -0.000000 0.000000
- joint right_shoulder_Z: origin xyz=0.022196 -0.038116 -0.104014 rpy=0.000000 -0.000000 0.000000 -> xyz=0.001037 -0.058602 0.168760 rpy=0.000000 -0.000000 0.000000
- joint right_wrist_Z: origin xyz=0.000000 -0.156657 0.000000 rpy=0.000000 -0.000000 0.000000 -> xyz=0.000000 -0.264197 0.000000 rpy=0.000000 -0.000000 0.000000
