Commit message: need to be tested for the collision capsules in rviz

File: urdf/human_scaled.urdf (robot description, URDF)
Before this commit: robot human_scaled, 80 links, 79 joints
Joints:
- joint joint_C7: origin xyz=-0.088296 0.568608 0.022895 rpy=0.000000 -0.000000 0.000000 -> xyz=-0.100611 0.567192 0.025482 rpy=0.000000 -0.000000 0.000000
- joint joint_Head: origin xyz=-0.063170 0.190906 -0.017908 rpy=0.000000 -0.000000 0.000000 -> xyz=-0.063930 0.201538 -0.024791 rpy=0.000000 -0.000000 0.000000
- joint joint_L5MHD: origin xyz=0.149075 -0.028134 0.077726 rpy=0.000000 -0.000000 0.000000 -> xyz=0.139112 -0.032538 0.070445 rpy=0.000000 -0.000000 0.000000
- joint joint_LANK: origin xyz=0.020762 -0.408001 -0.021350 rpy=0.000000 -0.000000 0.000000 -> xyz=0.017679 -0.395764 -0.023584 rpy=0.000000 -0.000000 0.000000
- joint joint_LASI: origin xyz=-0.032298 0.225521 0.042993 rpy=0.000000 -0.000000 0.000000 -> xyz=-0.001515 0.242680 0.029730 rpy=0.000000 -0.000000 0.000000
- joint joint_LELB: origin xyz=0.005704 -0.316023 -0.013916 rpy=0.000000 -0.000000 0.000000 -> xyz=-0.006837 -0.317514 -0.029231 rpy=0.000000 -0.000000 0.000000
- joint joint_LEar: origin xyz=-0.014424 0.067292 -0.069737 rpy=0.000000 -0.000000 0.000000 -> xyz=-0.016425 0.065153 -0.069736 rpy=0.000000 -0.000000 0.000000
- joint joint_LEye: origin xyz=0.073003 0.141644 -0.056717 rpy=0.000000 -0.000000 0.000000 -> xyz=0.063552 0.132560 -0.068608 rpy=0.000000 -0.000000 0.000000
- joint joint_LHEE: origin xyz=-0.241040 -0.036928 0.119340 rpy=0.000000 -0.000000 0.000000 -> xyz=-0.278009 -0.041094 0.118821 rpy=0.000000 -0.000000 0.000000
- joint joint_LKNE: origin xyz=0.010368 -0.359988 -0.049023 rpy=0.000000 -0.000000 0.000000 -> xyz=0.011890 -0.356177 -0.039188 rpy=0.000000 -0.000000 0.000000
- joint joint_LMANK: origin xyz=-0.023774 -0.406030 0.031546 rpy=0.000000 -0.000000 0.000000 -> xyz=-0.024057 -0.398057 0.033115 rpy=0.000000 -0.000000 0.000000
- joint joint_LMELB: origin xyz=-0.033072 -0.327266 0.067426 rpy=0.000000 -0.000000 0.000000 -> xyz=-0.010889 -0.328254 0.038482 rpy=0.000000 -0.000000 0.000000
- joint joint_LMID: origin xyz=0.000859 -0.151239 -0.000883 rpy=0.000000 -0.000000 0.000000 -> xyz=0.001608 -0.161306 0.000365 rpy=0.000000 -0.000000 0.000000
- joint joint_LMKNE: origin xyz=-0.063080 -0.290571 0.011084 rpy=0.000000 -0.000000 0.000000 -> xyz=-0.058133 -0.282974 0.016576 rpy=0.000000 -0.000000 0.000000
- joint joint_LMWRI: origin xyz=-0.013293 -0.286383 0.026804 rpy=0.000000 -0.000000 0.000000 -> xyz=-0.004872 -0.288360 0.025225 rpy=0.000000 -0.000000 0.000000
- joint joint_LPIN: origin xyz=0.013130 -0.166097 0.060680 rpy=0.000000 -0.000000 0.000000 -> xyz=0.018336 -0.168711 0.038496 rpy=0.000000 -0.000000 0.000000
- joint joint_LPSI: origin xyz=-0.184575 0.087863 0.019108 rpy=0.000000 -0.000000 0.000000 -> xyz=-0.167189 0.123759 0.007132 rpy=0.000000 -0.000000 0.000000
- joint joint_LSHO: origin xyz=0.006880 -0.041848 -0.155752 rpy=0.000000 -0.000000 0.000000 -> xyz=-0.001345 -0.035280 -0.151045 rpy=0.000000 -0.000000 0.000000
- joint joint_LTHU: origin xyz=0.001630 -0.133798 -0.067962 rpy=0.000000 -0.000000 0.000000 -> xyz=0.003558 -0.150337 -0.041916 rpy=0.000000 -0.000000 0.000000
- joint joint_LTOE: origin xyz=0.134847 -0.045692 0.155654 rpy=0.000000 -0.000000 0.000000 -> xyz=0.127206 -0.045869 0.147680 rpy=0.000000 -0.000000 0.000000
- joint joint_LWRI: origin xyz=-0.012270 -0.278828 -0.031263 rpy=0.000000 -0.000000 0.000000 -> xyz=-0.004754 -0.277855 -0.009353 rpy=0.000000 -0.000000 0.000000
- joint joint_Nose: origin xyz=0.125446 0.128348 -0.023599 rpy=0.000000 -0.000000 0.000000 -> xyz=0.115885 0.117941 -0.038805 rpy=0.000000 -0.000000 0.000000
- joint joint_R5MHD: origin xyz=0.157476 -0.035910 -0.043982 rpy=0.000000 -0.000000 0.000000 -> xyz=0.155558 -0.021142 -0.058071 rpy=0.000000 -0.000000 0.000000
- joint joint_RANK: origin xyz=0.017420 -0.398158 0.034951 rpy=0.000000 -0.000000 0.000000 -> xyz=0.014759 -0.389808 0.036887 rpy=0.000000 -0.000000 0.000000
- joint joint_RASI: origin xyz=0.023423 0.026316 0.173711 rpy=0.000000 -0.000000 0.000000 -> xyz=0.011669 0.030216 0.157205 rpy=0.000000 -0.000000 0.000000
- joint joint_RELB: origin xyz=-0.014785 -0.320281 0.032681 rpy=0.000000 -0.000000 0.000000 -> xyz=-0.015808 -0.333866 0.034943 rpy=0.000000 -0.000000 0.000000
- joint joint_REar: origin xyz=-0.004108 0.096011 0.084225 rpy=0.000000 -0.000000 0.000000 -> xyz=-0.001458 0.108347 0.085418 rpy=0.000000 -0.000000 0.000000
- joint joint_REye: origin xyz=0.075094 0.151108 0.013567 rpy=0.000000 -0.000000 0.000000 -> xyz=0.068544 0.152463 -0.001137 rpy=0.000000 -0.000000 0.000000
- joint joint_RHEE: origin xyz=-0.254177 -0.034181 -0.110385 rpy=0.000000 -0.000000 0.000000 -> xyz=-0.271050 -0.023819 -0.127330 rpy=0.000000 -0.000000 0.000000
- joint joint_RKNE: origin xyz=0.010147 -0.379736 0.016104 rpy=0.000000 -0.000000 0.000000 -> xyz=0.016350 -0.363043 0.005955 rpy=0.000000 -0.000000 0.000000
- joint joint_RMANK: origin xyz=-0.009697 -0.403449 -0.031248 rpy=0.000000 -0.000000 0.000000 -> xyz=-0.009884 -0.392544 -0.028441 rpy=0.000000 -0.000000 0.000000
- joint joint_RMELB: origin xyz=-0.029558 -0.327197 -0.052072 rpy=0.000000 -0.000000 0.000000 -> xyz=-0.040618 -0.340451 -0.053799 rpy=0.000000 -0.000000 0.000000
- joint joint_RMID: origin xyz=0.001853 -0.176359 0.000040 rpy=0.000000 -0.000000 0.000000 -> xyz=0.001716 -0.159929 0.000714 rpy=0.000000 -0.000000 0.000000
- joint joint_RMKNE: origin xyz=-0.074963 -0.393659 -0.068235 rpy=0.000000 -0.000000 0.000000 -> xyz=-0.068569 -0.373145 -0.076798 rpy=0.000000 -0.000000 0.000000
- joint joint_RMWRI: origin xyz=-0.010818 -0.311185 -0.018371 rpy=0.000000 -0.000000 0.000000 -> xyz=-0.013497 -0.308934 -0.017701 rpy=0.000000 -0.000000 0.000000
- joint joint_RPIN: origin xyz=0.009811 -0.190681 -0.040969 rpy=0.000000 -0.000000 0.000000 -> xyz=0.011655 -0.168876 -0.031495 rpy=0.000000 -0.000000 0.000000
- joint joint_RPSI: origin xyz=-0.151028 -0.003926 0.083364 rpy=0.000000 -0.000000 0.000000 -> xyz=-0.156804 0.020757 0.070160 rpy=0.000000 -0.000000 0.000000
- joint joint_RSHO: origin xyz=-0.038804 -0.004832 0.216822 rpy=0.000000 -0.000000 0.000000 -> xyz=-0.040225 -0.010422 0.222584 rpy=0.000000 -0.000000 0.000000
- joint joint_RTHU: origin xyz=0.006359 -0.148331 0.039116 rpy=0.000000 -0.000000 0.000000 -> xyz=0.008049 -0.138548 0.036967 rpy=0.000000 -0.000000 0.000000
- joint joint_RTOE: origin xyz=0.169712 -0.037041 -0.150108 rpy=0.000000 -0.000000 0.000000 -> xyz=0.176854 -0.023563 -0.171505 rpy=0.000000 -0.000000 0.000000
- joint joint_RWRI: origin xyz=-0.010523 -0.299224 0.016849 rpy=0.000000 -0.000000 0.000000 -> xyz=-0.012556 -0.303122 0.015176 rpy=0.000000 -0.000000 0.000000
- joint joint_T11: origin xyz=-0.168156 0.274745 0.230525 rpy=0.000000 -0.000000 0.000000 -> xyz=-0.174368 0.264446 0.233544 rpy=0.000000 -0.000000 0.000000
- joint joint_T6: origin xyz=-0.126739 0.420060 0.028283 rpy=0.000000 -0.000000 0.000000 -> xyz=-0.134151 0.416844 0.025824 rpy=0.000000 -0.000000 0.000000
- joint left_ankle_Z: origin xyz=0.000000 -0.438307 0.000000 rpy=0.000000 -0.000000 0.000000 -> xyz=0.000000 -0.422383 0.000000 rpy=0.000000 -0.000000 0.000000
- joint left_clavicle_joint_X: origin xyz=0.000000 0.618421 0.000000 rpy=0.000000 -0.000000 0.000000 -> xyz=0.000000 0.618201 0.000000 rpy=0.000000 -0.000000 0.000000
- joint left_elbow_Z: origin xyz=0.000000 -0.288015 0.000000 rpy=0.000000 -0.000000 0.000000 -> xyz=0.000000 -0.287992 0.000000 rpy=0.000000 -0.000000 0.000000
- joint left_hip_Z: origin xyz=0.022765 -0.090673 -0.088195 rpy=0.000000 -0.000000 0.000000 -> xyz=0.019157 -0.091987 -0.089385 rpy=0.000000 -0.000000 0.000000
- joint left_knee_Z: origin xyz=0.000000 -0.395648 0.000000 rpy=0.000000 -0.000000 0.000000 -> xyz=0.000000 -0.386267 0.000000 rpy=0.000000 -0.000000 0.000000
- joint left_shoulder_Z: origin xyz=-0.001037 -0.056159 -0.168760 rpy=0.000000 -0.000000 0.000000 -> xyz=-0.002709 -0.049405 -0.168645 rpy=0.000000 -0.000000 0.000000
- joint left_wrist_Z: origin xyz=0.000000 -0.256851 0.000000 rpy=0.000000 -0.000000 0.000000 -> xyz=0.000000 -0.249688 0.000000 rpy=0.000000 -0.000000 0.000000
- joint middle_cervical_Z: origin xyz=0.000000 0.642803 0.000000 rpy=0.000000 -0.000000 0.000000 -> xyz=0.000000 0.640758 0.000000 rpy=0.000000 -0.000000 0.000000
- joint middle_thoracic_Z: origin xyz=0.000000 0.146114 0.000000 rpy=0.000000 -0.000000 0.000000 -> xyz=0.000000 0.146444 0.000000 rpy=0.000000 -0.000000 0.000000
- joint right_ankle_Z: origin xyz=0.000000 -0.418762 0.000000 rpy=0.000000 -0.000000 0.000000 -> xyz=0.000000 -0.417070 0.000000 rpy=0.000000 -0.000000 0.000000
- joint right_clavicle_joint_X: origin xyz=0.000000 0.618421 0.000000 rpy=0.000000 -0.000000 0.000000 -> xyz=0.000000 0.618201 0.000000 rpy=0.000000 -0.000000 0.000000
- joint right_elbow_Z: origin xyz=0.000000 -0.274470 0.000000 rpy=0.000000 -0.000000 0.000000 -> xyz=0.000000 -0.285602 0.000000 rpy=0.000000 -0.000000 0.000000
- joint right_hip_Z: origin xyz=0.022765 -0.090400 0.088474 rpy=0.000000 -0.000000 0.000000 -> xyz=0.019157 -0.091623 0.089758 rpy=0.000000 -0.000000 0.000000
- joint right_knee_Z: origin xyz=0.000000 -0.402147 0.000000 rpy=0.000000 -0.000000 0.000000 -> xyz=0.000000 -0.391118 0.000000 rpy=0.000000 -0.000000 0.000000
- joint right_shoulder_Z: origin xyz=0.001037 -0.058602 0.168760 rpy=0.000000 -0.000000 0.000000 -> xyz=0.002709 -0.065418 0.168645 rpy=0.000000 -0.000000 0.000000
- joint right_wrist_Z: origin xyz=0.000000 -0.264197 0.000000 rpy=0.000000 -0.000000 0.000000 -> xyz=0.000000 -0.273434 0.000000 rpy=0.000000 -0.000000 0.000000

Commit message: reapply the right world transform

File: urdf/human_scaled.urdf (robot description, URDF)
Before this commit: robot human_scaled, 80 links, 79 joints
Joints:
- joint joint_C7: origin xyz=-0.100611 0.567192 0.025482 rpy=0.000000 -0.000000 0.000000 -> xyz=-0.096710 0.359146 -0.004305 rpy=0.000000 -0.000000 0.000000
- joint joint_Head: origin xyz=-0.063930 0.201538 -0.024791 rpy=0.000000 -0.000000 0.000000 -> xyz=-0.041991 0.273084 -0.017392 rpy=0.000000 -0.000000 0.000000
- joint joint_L5MHD: origin xyz=0.139112 -0.032538 0.070445 rpy=0.000000 -0.000000 0.000000 -> xyz=0.157470 -0.039389 -0.036140 rpy=0.000000 -0.000000 0.000000
- joint joint_LANK: origin xyz=0.017679 -0.395764 -0.023584 rpy=0.000000 -0.000000 0.000000 -> xyz=-0.004963 -0.425956 -0.033529 rpy=0.000000 -0.000000 0.000000
- joint joint_LASI: origin xyz=-0.001515 0.242680 0.029730 rpy=0.000000 -0.000000 0.000000 -> xyz=0.102085 -0.001730 -0.123978 rpy=0.000000 -0.000000 0.000000
- joint joint_LELB: origin xyz=-0.006837 -0.317514 -0.029231 rpy=0.000000 -0.000000 0.000000 -> xyz=0.016517 -0.281298 -0.021844 rpy=0.000000 -0.000000 0.000000
- joint joint_LEar: origin xyz=-0.016425 0.065153 -0.069736 rpy=0.000000 -0.000000 0.000000 -> xyz=-0.022314 0.151849 -0.091175 rpy=0.000000 -0.000000 0.000000
- joint joint_LEye: origin xyz=0.063552 0.132560 -0.068608 rpy=0.000000 -0.000000 0.000000 -> xyz=0.080435 0.194143 -0.067381 rpy=0.000000 -0.000000 0.000000
- joint joint_LHEE: origin xyz=-0.278009 -0.041094 0.118821 rpy=0.000000 -0.000000 0.000000 -> xyz=-0.062248 -0.037052 0.009649 rpy=0.000000 -0.000000 0.000000
- joint joint_LKNE: origin xyz=0.011890 -0.356177 -0.039188 rpy=0.000000 -0.000000 0.000000 -> xyz=0.018451 -0.393216 -0.049664 rpy=0.000000 -0.000000 0.000000
- joint joint_LMANK: origin xyz=-0.024057 -0.398057 0.033115 rpy=0.000000 -0.000000 0.000000 -> xyz=0.004838 -0.425554 0.034737 rpy=0.000000 -0.000000 0.000000
- joint joint_LMELB: origin xyz=-0.010889 -0.328254 0.038482 rpy=0.000000 -0.000000 0.000000 -> xyz=-0.013743 -0.289900 0.052378 rpy=0.000000 -0.000000 0.000000
- joint joint_LMID: origin xyz=0.001608 -0.161306 0.000365 rpy=0.000000 -0.000000 0.000000 -> xyz=0.000134 -0.127651 -0.000134 rpy=0.000000 -0.000000 0.000000
- joint joint_LMKNE: origin xyz=-0.058133 -0.282974 0.016576 rpy=0.000000 -0.000000 0.000000 -> xyz=-0.017656 -0.390435 0.060327 rpy=0.000000 -0.000000 0.000000
- joint joint_LMWRI: origin xyz=-0.004872 -0.288360 0.025225 rpy=0.000000 -0.000000 0.000000 -> xyz=-0.007869 -0.254794 0.014894 rpy=0.000000 -0.000000 0.000000
- joint joint_LPIN: origin xyz=0.018336 -0.168711 0.038496 rpy=0.000000 -0.000000 0.000000 -> xyz=0.008008 -0.139439 0.035844 rpy=0.000000 -0.000000 0.000000
- joint joint_LPSI: origin xyz=-0.167189 0.123759 0.007132 rpy=0.000000 -0.000000 0.000000 -> xyz=-0.080733 -0.001011 -0.061404 rpy=0.000000 -0.000000 0.000000
- joint joint_LSHO: origin xyz=-0.001345 -0.035280 -0.151045 rpy=0.000000 -0.000000 0.000000 -> xyz=-0.033860 0.007994 -0.169985 rpy=0.000000 -0.000000 0.000000
- joint joint_LTHU: origin xyz=0.003558 -0.150337 -0.041916 rpy=0.000000 -0.000000 0.000000 -> xyz=0.002554 -0.105806 -0.037263 rpy=0.000000 -0.000000 0.000000
- joint joint_LTOE: origin xyz=0.127206 -0.045869 0.147680 rpy=0.000000 -0.000000 0.000000 -> xyz=0.194308 -0.035284 0.024519 rpy=0.000000 -0.000000 0.000000
- joint joint_LWRI: origin xyz=-0.004754 -0.277855 -0.009353 rpy=0.000000 -0.000000 0.000000 -> xyz=-0.008271 -0.244469 -0.015124 rpy=0.000000 -0.000000 0.000000
- joint joint_Nose: origin xyz=0.115885 0.117941 -0.038805 rpy=0.000000 -0.000000 0.000000 -> xyz=0.142573 0.162561 -0.044137 rpy=0.000000 -0.000000 0.000000
- joint joint_R5MHD: origin xyz=0.155558 -0.021142 -0.058071 rpy=0.000000 -0.000000 0.000000 -> xyz=0.135414 -0.057873 0.039116 rpy=0.000000 -0.000000 0.000000
- joint joint_RANK: origin xyz=0.014759 -0.389808 0.036887 rpy=0.000000 -0.000000 0.000000 -> xyz=-0.008165 -0.430777 0.031667 rpy=0.000000 -0.000000 0.000000
- joint joint_RASI: origin xyz=0.011669 0.030216 0.157205 rpy=0.000000 -0.000000 0.000000 -> xyz=0.071653 -0.003039 0.119173 rpy=0.000000 -0.000000 0.000000
- joint joint_RELB: origin xyz=-0.015808 -0.333866 0.034943 rpy=0.000000 -0.000000 0.000000 -> xyz=0.021001 -0.271890 0.019195 rpy=0.000000 -0.000000 0.000000
- joint joint_REar: origin xyz=-0.001458 0.108347 0.085418 rpy=0.000000 -0.000000 0.000000 -> xyz=-0.018888 0.153909 0.063930 rpy=0.000000 -0.000000 0.000000
- joint joint_REye: origin xyz=0.068544 0.152463 -0.001137 rpy=0.000000 -0.000000 0.000000 -> xyz=0.086966 0.196285 -0.000524 rpy=0.000000 -0.000000 0.000000
- joint joint_RHEE: origin xyz=-0.271050 -0.023819 -0.127330 rpy=0.000000 -0.000000 0.000000 -> xyz=-0.059978 -0.049045 -0.006712 rpy=0.000000 -0.000000 0.000000
- joint joint_RKNE: origin xyz=0.016350 -0.363043 0.005955 rpy=0.000000 -0.000000 0.000000 -> xyz=0.009430 -0.402697 0.059176 rpy=0.000000 -0.000000 0.000000
- joint joint_RMANK: origin xyz=-0.009884 -0.392544 -0.028441 rpy=0.000000 -0.000000 0.000000 -> xyz=0.007484 -0.429894 -0.035522 rpy=0.000000 -0.000000 0.000000
- joint joint_RMELB: origin xyz=-0.040618 -0.340451 -0.053799 rpy=0.000000 -0.000000 0.000000 -> xyz=-0.017321 -0.290598 -0.050701 rpy=0.000000 -0.000000 0.000000
- joint joint_RMID: origin xyz=0.001716 -0.159929 0.000714 rpy=0.000000 -0.000000 0.000000 -> xyz=0.000312 -0.147366 0.000153 rpy=0.000000 -0.000000 0.000000
- joint joint_RMKNE: origin xyz=-0.068569 -0.373145 -0.076798 rpy=0.000000 -0.000000 0.000000 -> xyz=-0.009362 -0.399484 -0.054978 rpy=0.000000 -0.000000 0.000000
- joint joint_RMWRI: origin xyz=-0.013497 -0.308934 -0.017701 rpy=0.000000 -0.000000 0.000000 -> xyz=-0.006950 -0.264701 -0.014304 rpy=0.000000 -0.000000 0.000000
- joint joint_RPIN: origin xyz=0.011655 -0.168876 -0.031495 rpy=0.000000 -0.000000 0.000000 -> xyz=0.006499 -0.165417 -0.032417 rpy=0.000000 -0.000000 0.000000
- joint joint_RPSI: origin xyz=-0.156804 0.020757 0.070160 rpy=0.000000 -0.000000 0.000000 -> xyz=-0.090305 -0.002493 0.057887 rpy=0.000000 -0.000000 0.000000
- joint joint_RSHO: origin xyz=-0.040225 -0.010422 0.222584 rpy=0.000000 -0.000000 0.000000 -> xyz=-0.024866 -0.002624 0.162821 rpy=0.000000 -0.000000 0.000000
- joint joint_RTHU: origin xyz=0.008049 -0.138548 0.036967 rpy=0.000000 -0.000000 0.000000 -> xyz=0.005131 -0.109165 0.025781 rpy=0.000000 -0.000000 0.000000
- joint joint_RTOE: origin xyz=0.176854 -0.023563 -0.171505 rpy=0.000000 -0.000000 0.000000 -> xyz=0.215748 -0.035263 -0.038456 rpy=0.000000 -0.000000 0.000000
- joint joint_RWRI: origin xyz=-0.012556 -0.303122 0.015176 rpy=0.000000 -0.000000 0.000000 -> xyz=-0.008032 -0.258089 0.009991 rpy=0.000000 -0.000000 0.000000
- joint joint_T11: origin xyz=-0.174368 0.264446 0.233544 rpy=0.000000 -0.000000 0.000000 -> xyz=-0.138300 0.223500 -0.005480 rpy=0.000000 -0.000000 0.000000
- joint joint_T6: origin xyz=-0.134151 0.416844 0.025824 rpy=0.000000 -0.000000 0.000000 -> xyz=-0.135938 0.212609 -0.000873 rpy=0.000000 -0.000000 0.000000
- joint left_ankle_Z: origin xyz=0.000000 -0.422383 0.000000 rpy=0.000000 -0.000000 0.000000 -> xyz=0.000000 -0.424286 0.000000 rpy=0.000000 -0.000000 0.000000
- joint left_clavicle_joint_X: origin xyz=0.000000 0.618201 0.000000 rpy=0.000000 -0.000000 0.000000 -> xyz=0.000000 0.322987 0.000000 rpy=0.000000 -0.000000 0.000000
- joint left_elbow_Z: origin xyz=0.000000 -0.287992 0.000000 rpy=0.000000 -0.000000 0.000000 -> xyz=0.000000 -0.285890 0.000000 rpy=0.000000 -0.000000 0.000000
- joint left_hip_Z: origin xyz=0.019157 -0.091987 -0.089385 rpy=0.000000 -0.000000 0.000000 -> xyz=0.012680 -0.090869 -0.088258 rpy=0.000000 -0.000000 0.000000
- joint left_knee_Z: origin xyz=0.000000 -0.386267 0.000000 rpy=0.000000 -0.000000 0.000000 -> xyz=0.000000 -0.390262 0.000000 rpy=0.000000 -0.000000 0.000000
- joint left_shoulder_Z: origin xyz=-0.002709 -0.049405 -0.168645 rpy=0.000000 -0.000000 0.000000 -> xyz=-0.004767 -0.051810 -0.166418 rpy=0.000000 -0.000000 0.000000
- joint left_wrist_Z: origin xyz=0.000000 -0.249688 0.000000 rpy=0.000000 -0.000000 0.000000 -> xyz=0.000000 -0.250601 0.000000 rpy=0.000000 -0.000000 0.000000
- joint middle_cervical_Z: origin xyz=0.000000 0.640758 0.000000 rpy=0.000000 -0.000000 0.000000 -> xyz=0.000000 0.350217 0.000000 rpy=0.000000 -0.000000 0.000000
- joint middle_thoracic_Z: origin xyz=0.000000 0.146444 0.000000 rpy=0.000000 -0.000000 0.000000 -> xyz=0.000000 0.150477 0.000000 rpy=0.000000 -0.000000 0.000000
- joint right_ankle_Z: origin xyz=0.000000 -0.417070 0.000000 rpy=0.000000 -0.000000 0.000000 -> xyz=0.000000 -0.427762 0.000000 rpy=0.000000 -0.000000 0.000000
- joint right_clavicle_joint_X: origin xyz=0.000000 0.618201 0.000000 rpy=0.000000 -0.000000 0.000000 -> xyz=0.000000 0.322987 0.000000 rpy=0.000000 -0.000000 0.000000
- joint right_elbow_Z: origin xyz=0.000000 -0.285602 0.000000 rpy=0.000000 -0.000000 0.000000 -> xyz=0.000000 -0.282315 0.000000 rpy=0.000000 -0.000000 0.000000
- joint right_hip_Z: origin xyz=0.019157 -0.091623 0.089758 rpy=0.000000 -0.000000 0.000000 -> xyz=0.012680 -0.090469 0.088668 rpy=0.000000 -0.000000 0.000000
- joint right_knee_Z: origin xyz=0.000000 -0.391118 0.000000 rpy=0.000000 -0.000000 0.000000 -> xyz=0.000000 -0.398496 0.000000 rpy=0.000000 -0.000000 0.000000
- joint right_shoulder_Z: origin xyz=0.002709 -0.065418 0.168645 rpy=0.000000 -0.000000 0.000000 -> xyz=0.004767 -0.061449 0.166418 rpy=0.000000 -0.000000 0.000000
- joint right_wrist_Z: origin xyz=0.000000 -0.273434 0.000000 rpy=0.000000 -0.000000 0.000000 -> xyz=0.000000 -0.262820 0.000000 rpy=0.000000 -0.000000 0.000000
