Commit message: now it is working properly yay !

File: urdf/human_scaled.urdf (robot description, URDF)
Before this commit: robot human_scaled, 80 links, 79 joints
Joints:
- joint joint_C7: origin xyz=-0.096710 0.359146 -0.004305 rpy=0.000000 -0.000000 0.000000 -> xyz=-0.091198 0.361775 -0.002790 rpy=0.000000 -0.000000 0.000000
- joint joint_Head: origin xyz=-0.041991 0.273084 -0.017392 rpy=0.000000 -0.000000 0.000000 -> xyz=-0.046599 0.273714 -0.015816 rpy=0.000000 -0.000000 0.000000
- joint joint_L5MHD: origin xyz=0.157470 -0.039389 -0.036140 rpy=0.000000 -0.000000 0.000000 -> xyz=0.153851 -0.039208 -0.037582 rpy=0.000000 -0.000000 0.000000
- joint joint_LANK: origin xyz=-0.004963 -0.425956 -0.033529 rpy=0.000000 -0.000000 0.000000 -> xyz=-0.004681 -0.418416 -0.032406 rpy=0.000000 -0.000000 0.000000
- joint joint_LASI: origin xyz=0.102085 -0.001730 -0.123978 rpy=0.000000 -0.000000 0.000000 -> xyz=0.110483 -0.000420 -0.124143 rpy=0.000000 -0.000000 0.000000
- joint joint_LELB: origin xyz=0.016517 -0.281298 -0.021844 rpy=0.000000 -0.000000 0.000000 -> xyz=0.023642 -0.276717 -0.025527 rpy=0.000000 -0.000000 0.000000
- joint joint_LEar: origin xyz=-0.022314 0.151849 -0.091175 rpy=0.000000 -0.000000 0.000000 -> xyz=-0.015656 0.150988 -0.094927 rpy=0.000000 -0.000000 0.000000
- joint joint_LEye: origin xyz=0.080435 0.194143 -0.067381 rpy=0.000000 -0.000000 0.000000 -> xyz=0.076198 0.195533 -0.069980 rpy=0.000000 -0.000000 0.000000
- joint joint_LHEE: origin xyz=-0.062248 -0.037052 0.009649 rpy=0.000000 -0.000000 0.000000 -> xyz=-0.060434 -0.037705 0.006636 rpy=0.000000 -0.000000 0.000000
- joint joint_LKNE: origin xyz=0.018451 -0.393216 -0.049664 rpy=0.000000 -0.000000 0.000000 -> xyz=0.016755 -0.390184 -0.051785 rpy=0.000000 -0.000000 0.000000
- joint joint_LMANK: origin xyz=0.004838 -0.425554 0.034737 rpy=0.000000 -0.000000 0.000000 -> xyz=0.004620 -0.418749 0.034283 rpy=0.000000 -0.000000 0.000000
- joint joint_LMELB: origin xyz=-0.013743 -0.289900 0.052378 rpy=0.000000 -0.000000 0.000000 -> xyz=-0.021115 -0.293933 0.050511 rpy=0.000000 -0.000000 0.000000
- joint joint_LMID: origin xyz=0.000134 -0.127651 -0.000134 rpy=0.000000 -0.000000 0.000000 -> xyz=0.000057 -0.124926 -0.000088 rpy=0.000000 -0.000000 0.000000
- joint joint_LMKNE: origin xyz=-0.017656 -0.390435 0.060327 rpy=0.000000 -0.000000 0.000000 -> xyz=-0.016435 -0.388077 0.058989 rpy=0.000000 -0.000000 0.000000
- joint joint_LMWRI: origin xyz=-0.007869 -0.254794 0.014894 rpy=0.000000 -0.000000 0.000000 -> xyz=-0.007059 -0.261266 0.020606 rpy=0.000000 -0.000000 0.000000
- joint joint_LPIN: origin xyz=0.008008 -0.139439 0.035844 rpy=0.000000 -0.000000 0.000000 -> xyz=0.009680 -0.131675 0.041498 rpy=0.000000 -0.000000 0.000000
- joint joint_LPSI: origin xyz=-0.080733 -0.001011 -0.061404 rpy=0.000000 -0.000000 0.000000 -> xyz=-0.095666 -0.002203 -0.061033 rpy=0.000000 -0.000000 0.000000
- joint joint_LSHO: origin xyz=-0.033860 0.007994 -0.169985 rpy=0.000000 -0.000000 0.000000 -> xyz=-0.022357 0.008630 -0.171084 rpy=0.000000 -0.000000 0.000000
- joint joint_LTHU: origin xyz=0.002554 -0.105806 -0.037263 rpy=0.000000 -0.000000 0.000000 -> xyz=0.002713 -0.112238 -0.045777 rpy=0.000000 -0.000000 0.000000
- joint joint_LTOE: origin xyz=0.194308 -0.035284 0.024519 rpy=0.000000 -0.000000 0.000000 -> xyz=0.191646 -0.035637 0.023752 rpy=0.000000 -0.000000 0.000000
- joint joint_LWRI: origin xyz=-0.008271 -0.244469 -0.015124 rpy=0.000000 -0.000000 0.000000 -> xyz=-0.006815 -0.257132 -0.020921 rpy=0.000000 -0.000000 0.000000
- joint joint_Nose: origin xyz=0.142573 0.162561 -0.044137 rpy=0.000000 -0.000000 0.000000 -> xyz=0.127843 0.167673 -0.044920 rpy=0.000000 -0.000000 0.000000
- joint joint_R5MHD: origin xyz=0.135414 -0.057873 0.039116 rpy=0.000000 -0.000000 0.000000 -> xyz=0.141600 -0.053325 0.038101 rpy=0.000000 -0.000000 0.000000
- joint joint_RANK: origin xyz=-0.008165 -0.430777 0.031667 rpy=0.000000 -0.000000 0.000000 -> xyz=-0.007756 -0.424210 0.031188 rpy=0.000000 -0.000000 0.000000
- joint joint_RASI: origin xyz=0.071653 -0.003039 0.119173 rpy=0.000000 -0.000000 0.000000 -> xyz=0.087809 -0.002553 0.119786 rpy=0.000000 -0.000000 0.000000
- joint joint_RELB: origin xyz=0.021001 -0.271890 0.019195 rpy=0.000000 -0.000000 0.000000 -> xyz=0.022612 -0.272736 0.020869 rpy=0.000000 -0.000000 0.000000
- joint joint_REar: origin xyz=-0.018888 0.153909 0.063930 rpy=0.000000 -0.000000 0.000000 -> xyz=-0.011248 0.152764 0.062201 rpy=0.000000 -0.000000 0.000000
- joint joint_REye: origin xyz=0.086966 0.196285 -0.000524 rpy=0.000000 -0.000000 0.000000 -> xyz=0.080470 0.198005 -0.002001 rpy=0.000000 -0.000000 0.000000
- joint joint_RHEE: origin xyz=-0.059978 -0.049045 -0.006712 rpy=0.000000 -0.000000 0.000000 -> xyz=-0.059928 -0.046133 -0.009843 rpy=0.000000 -0.000000 0.000000
- joint joint_RKNE: origin xyz=0.009430 -0.402697 0.059176 rpy=0.000000 -0.000000 0.000000 -> xyz=0.012975 -0.394391 0.059017 rpy=0.000000 -0.000000 0.000000
- joint joint_RMANK: origin xyz=0.007484 -0.429894 -0.035522 rpy=0.000000 -0.000000 0.000000 -> xyz=0.007200 -0.425070 -0.036153 rpy=0.000000 -0.000000 0.000000
- joint joint_RMELB: origin xyz=-0.017321 -0.290598 -0.050701 rpy=0.000000 -0.000000 0.000000 -> xyz=-0.018450 -0.290948 -0.050178 rpy=0.000000 -0.000000 0.000000
- joint joint_RMID: origin xyz=0.000312 -0.147366 0.000153 rpy=0.000000 -0.000000 0.000000 -> xyz=0.000230 -0.137826 0.000073 rpy=0.000000 -0.000000 0.000000
- joint joint_RMKNE: origin xyz=-0.009362 -0.399484 -0.054978 rpy=0.000000 -0.000000 0.000000 -> xyz=-0.012901 -0.394067 -0.053650 rpy=0.000000 -0.000000 0.000000
- joint joint_RMWRI: origin xyz=-0.006950 -0.264701 -0.014304 rpy=0.000000 -0.000000 0.000000 -> xyz=-0.007465 -0.267498 -0.018388 rpy=0.000000 -0.000000 0.000000
- joint joint_RPIN: origin xyz=0.006499 -0.165417 -0.032417 rpy=0.000000 -0.000000 0.000000 -> xyz=0.007230 -0.142650 -0.037649 rpy=0.000000 -0.000000 0.000000
- joint joint_RPSI: origin xyz=-0.090305 -0.002493 0.057887 rpy=0.000000 -0.000000 0.000000 -> xyz=-0.100829 -0.002592 0.058275 rpy=0.000000 -0.000000 0.000000
- joint joint_RSHO: origin xyz=-0.024866 -0.002624 0.162821 rpy=0.000000 -0.000000 0.000000 -> xyz=-0.028144 -0.001419 0.165794 rpy=0.000000 -0.000000 0.000000
- joint joint_RTHU: origin xyz=0.005131 -0.109165 0.025781 rpy=0.000000 -0.000000 0.000000 -> xyz=0.006741 -0.114231 0.039600 rpy=0.000000 -0.000000 0.000000
- joint joint_RTOE: origin xyz=0.215748 -0.035263 -0.038456 rpy=0.000000 -0.000000 0.000000 -> xyz=0.214550 -0.035325 -0.038104 rpy=0.000000 -0.000000 0.000000
- joint joint_RWRI: origin xyz=-0.008032 -0.258089 0.009991 rpy=0.000000 -0.000000 0.000000 -> xyz=-0.007080 -0.265750 0.017250 rpy=0.000000 -0.000000 0.000000
- joint joint_T11: origin xyz=-0.138300 0.223500 -0.005480 rpy=0.000000 -0.000000 0.000000 -> xyz=-0.134230 0.226914 -0.005502 rpy=0.000000 -0.000000 0.000000
- joint joint_T6: origin xyz=-0.135938 0.212609 -0.000873 rpy=0.000000 -0.000000 0.000000 -> xyz=-0.135257 0.214055 0.000164 rpy=0.000000 -0.000000 0.000000
- joint left_ankle_Z: origin xyz=0.000000 -0.424286 0.000000 rpy=0.000000 -0.000000 0.000000 -> xyz=0.000000 -0.417170 0.000000 rpy=0.000000 -0.000000 0.000000
- joint left_clavicle_joint_X: origin xyz=0.000000 0.322987 0.000000 rpy=0.000000 -0.000000 0.000000 -> xyz=0.000000 0.326014 0.000000 rpy=0.000000 -0.000000 0.000000
- joint left_elbow_Z: origin xyz=0.000000 -0.285890 0.000000 rpy=0.000000 -0.000000 0.000000 -> xyz=0.000000 -0.285475 0.000000 rpy=0.000000 -0.000000 0.000000
- joint left_hip_Z: origin xyz=0.012680 -0.090869 -0.088258 rpy=0.000000 -0.000000 0.000000 -> xyz=0.025202 -0.090493 -0.088598 rpy=0.000000 -0.000000 0.000000
- joint left_knee_Z: origin xyz=0.000000 -0.390262 0.000000 rpy=0.000000 -0.000000 0.000000 -> xyz=0.000000 -0.387698 0.000000 rpy=0.000000 -0.000000 0.000000
- joint left_shoulder_Z: origin xyz=-0.004767 -0.051810 -0.166418 rpy=0.000000 -0.000000 0.000000 -> xyz=0.003712 -0.054580 -0.168501 rpy=0.000000 -0.000000 0.000000
- joint left_wrist_Z: origin xyz=0.000000 -0.250601 0.000000 rpy=0.000000 -0.000000 0.000000 -> xyz=0.000000 -0.259369 0.000000 rpy=0.000000 -0.000000 0.000000
- joint middle_cervical_Z: origin xyz=0.000000 0.350217 0.000000 rpy=0.000000 -0.000000 0.000000 -> xyz=0.000000 0.354247 0.000000 rpy=0.000000 -0.000000 0.000000
- joint middle_thoracic_Z: origin xyz=0.000000 0.150477 0.000000 rpy=0.000000 -0.000000 0.000000 -> xyz=0.000000 0.150702 0.000000 rpy=0.000000 -0.000000 0.000000
- joint right_ankle_Z: origin xyz=0.000000 -0.427762 0.000000 rpy=0.000000 -0.000000 0.000000 -> xyz=0.000000 -0.422321 0.000000 rpy=0.000000 -0.000000 0.000000
- joint right_clavicle_joint_X: origin xyz=0.000000 0.322987 0.000000 rpy=0.000000 -0.000000 0.000000 -> xyz=0.000000 0.326014 0.000000 rpy=0.000000 -0.000000 0.000000
- joint right_elbow_Z: origin xyz=0.000000 -0.282315 0.000000 rpy=0.000000 -0.000000 0.000000 -> xyz=0.000000 -0.282755 0.000000 rpy=0.000000 -0.000000 0.000000
- joint right_hip_Z: origin xyz=0.012680 -0.090469 0.088668 rpy=0.000000 -0.000000 0.000000 -> xyz=0.025202 -0.090799 0.088284 rpy=0.000000 -0.000000 0.000000
- joint right_knee_Z: origin xyz=0.000000 -0.398496 0.000000 rpy=0.000000 -0.000000 0.000000 -> xyz=0.000000 -0.391877 0.000000 rpy=0.000000 -0.000000 0.000000
- joint right_shoulder_Z: origin xyz=0.004767 -0.061449 0.166418 rpy=0.000000 -0.000000 0.000000 -> xyz=-0.003712 -0.060044 0.168501 rpy=0.000000 -0.000000 0.000000
- joint right_wrist_Z: origin xyz=0.000000 -0.262820 0.000000 rpy=0.000000 -0.000000 0.000000 -> xyz=0.000000 -0.267516 0.000000 rpy=0.000000 -0.000000 0.000000

Commit message: pose instead of markers ?

File: urdf/human_scaled.urdf (robot description, URDF)
Before this commit: robot human_scaled, 80 links, 79 joints
Joints:
- joint joint_C7: origin xyz=-0.091198 0.361775 -0.002790 rpy=0.000000 -0.000000 0.000000 -> xyz=-0.099200 0.343685 0.007565 rpy=0.000000 -0.000000 0.000000
- joint joint_Head: origin xyz=-0.046599 0.273714 -0.015816 rpy=0.000000 -0.000000 0.000000 -> xyz=-0.037045 0.265947 -0.003309 rpy=0.000000 -0.000000 0.000000
- joint joint_L5MHD: origin xyz=0.153851 -0.039208 -0.037582 rpy=0.000000 -0.000000 0.000000 -> xyz=0.152476 -0.044943 -0.041387 rpy=0.000000 -0.000000 0.000000
- joint joint_LANK: origin xyz=-0.004681 -0.418416 -0.032406 rpy=0.000000 -0.000000 0.000000 -> xyz=-0.004114 -0.437364 -0.030383 rpy=0.000000 -0.000000 0.000000
- joint joint_LASI: origin xyz=0.110483 -0.000420 -0.124143 rpy=0.000000 -0.000000 0.000000 -> xyz=0.096046 0.000442 -0.119931 rpy=0.000000 -0.000000 0.000000
- joint joint_LELB: origin xyz=0.023642 -0.276717 -0.025527 rpy=0.000000 -0.000000 0.000000 -> xyz=0.020817 -0.278353 -0.022552 rpy=0.000000 -0.000000 0.000000
- joint joint_LEar: origin xyz=-0.015656 0.150988 -0.094927 rpy=0.000000 -0.000000 0.000000 -> xyz=-0.019141 0.141001 -0.077093 rpy=0.000000 -0.000000 0.000000
- joint joint_LEye: origin xyz=0.076198 0.195533 -0.069980 rpy=0.000000 -0.000000 0.000000 -> xyz=0.100696 0.165863 -0.047471 rpy=0.000000 -0.000000 0.000000
- joint joint_LHEE: origin xyz=-0.060434 -0.037705 0.006636 rpy=0.000000 -0.000000 0.000000 -> xyz=-0.064002 -0.041486 0.005135 rpy=0.000000 -0.000000 0.000000
- joint joint_LKNE: origin xyz=0.016755 -0.390184 -0.051785 rpy=0.000000 -0.000000 0.000000 -> xyz=0.018240 -0.400951 -0.055369 rpy=0.000000 -0.000000 0.000000
- joint joint_LMANK: origin xyz=0.004620 -0.418749 0.034283 rpy=0.000000 -0.000000 0.000000 -> xyz=0.004044 -0.435735 0.035388 rpy=0.000000 -0.000000 0.000000
- joint joint_LMELB: origin xyz=-0.021115 -0.293933 0.050511 rpy=0.000000 -0.000000 0.000000 -> xyz=-0.017899 -0.293941 0.052578 rpy=0.000000 -0.000000 0.000000
- joint joint_LMID: origin xyz=0.000057 -0.124926 -0.000088 rpy=0.000000 -0.000000 0.000000 -> xyz=0.000072 -0.121823 -0.000218 rpy=0.000000 -0.000000 0.000000
- joint joint_LMKNE: origin xyz=-0.016435 -0.388077 0.058989 rpy=0.000000 -0.000000 0.000000 -> xyz=-0.018009 -0.399728 0.053041 rpy=0.000000 -0.000000 0.000000
- joint joint_LMWRI: origin xyz=-0.007059 -0.261266 0.020606 rpy=0.000000 -0.000000 0.000000 -> xyz=-0.008673 -0.255701 0.020159 rpy=0.000000 -0.000000 0.000000
- joint joint_LPIN: origin xyz=0.009680 -0.131675 0.041498 rpy=0.000000 -0.000000 0.000000 -> xyz=0.008471 -0.144385 0.052178 rpy=0.000000 -0.000000 0.000000
- joint joint_LPSI: origin xyz=-0.095666 -0.002203 -0.061033 rpy=0.000000 -0.000000 0.000000 -> xyz=-0.085300 -0.004126 -0.056365 rpy=0.000000 -0.000000 0.000000
- joint joint_LSHO: origin xyz=-0.022357 0.008630 -0.171084 rpy=0.000000 -0.000000 0.000000 -> xyz=-0.038838 0.006150 -0.162456 rpy=0.000000 -0.000000 0.000000
- joint joint_LTHU: origin xyz=0.002713 -0.112238 -0.045777 rpy=0.000000 -0.000000 0.000000 -> xyz=0.004512 -0.091306 -0.055733 rpy=0.000000 -0.000000 0.000000
- joint joint_LTOE: origin xyz=0.191646 -0.035637 0.023752 rpy=0.000000 -0.000000 0.000000 -> xyz=0.198641 -0.035147 0.023752 rpy=0.000000 -0.000000 0.000000
- joint joint_LWRI: origin xyz=-0.006815 -0.257132 -0.020921 rpy=0.000000 -0.000000 0.000000 -> xyz=-0.007653 -0.245097 -0.021676 rpy=0.000000 -0.000000 0.000000
- joint joint_Nose: origin xyz=0.127843 0.167673 -0.044920 rpy=0.000000 -0.000000 0.000000 -> xyz=0.149182 0.129668 -0.022498 rpy=0.000000 -0.000000 0.000000
- joint joint_R5MHD: origin xyz=0.141600 -0.053325 0.038101 rpy=0.000000 -0.000000 0.000000 -> xyz=0.141127 -0.057036 0.040700 rpy=0.000000 -0.000000 0.000000
- joint joint_RANK: origin xyz=-0.007756 -0.424210 0.031188 rpy=0.000000 -0.000000 0.000000 -> xyz=-0.003248 -0.441391 0.031198 rpy=0.000000 -0.000000 0.000000
- joint joint_RASI: origin xyz=0.087809 -0.002553 0.119786 rpy=0.000000 -0.000000 0.000000 -> xyz=0.091055 0.001004 0.117854 rpy=0.000000 -0.000000 0.000000
- joint joint_RELB: origin xyz=0.022612 -0.272736 0.020869 rpy=0.000000 -0.000000 0.000000 -> xyz=0.024132 -0.267544 0.021595 rpy=0.000000 -0.000000 0.000000
- joint joint_REar: origin xyz=-0.011248 0.152764 0.062201 rpy=0.000000 -0.000000 0.000000 -> xyz=-0.016668 0.144907 0.072865 rpy=0.000000 -0.000000 0.000000
- joint joint_REye: origin xyz=0.080470 0.198005 -0.002001 rpy=0.000000 -0.000000 0.000000 -> xyz=0.098913 0.168377 0.015136 rpy=0.000000 -0.000000 0.000000
- joint joint_RHEE: origin xyz=-0.059928 -0.046133 -0.009843 rpy=0.000000 -0.000000 0.000000 -> xyz=-0.057636 -0.045291 -0.011545 rpy=0.000000 -0.000000 0.000000
- joint joint_RKNE: origin xyz=0.012975 -0.394391 0.059017 rpy=0.000000 -0.000000 0.000000 -> xyz=0.008091 -0.408566 0.059432 rpy=0.000000 -0.000000 0.000000
- joint joint_RMANK: origin xyz=0.007200 -0.425070 -0.036153 rpy=0.000000 -0.000000 0.000000 -> xyz=0.005676 -0.441949 -0.036535 rpy=0.000000 -0.000000 0.000000
- joint joint_RMELB: origin xyz=-0.018450 -0.290948 -0.050178 rpy=0.000000 -0.000000 0.000000 -> xyz=-0.020245 -0.285325 -0.057262 rpy=0.000000 -0.000000 0.000000
- joint joint_RMID: origin xyz=0.000230 -0.137826 0.000073 rpy=0.000000 -0.000000 0.000000 -> xyz=0.000499 -0.133794 0.000161 rpy=0.000000 -0.000000 0.000000
- joint joint_RMKNE: origin xyz=-0.012901 -0.394067 -0.053650 rpy=0.000000 -0.000000 0.000000 -> xyz=-0.022023 -0.407247 -0.053934 rpy=0.000000 -0.000000 0.000000
- joint joint_RMWRI: origin xyz=-0.007465 -0.267498 -0.018388 rpy=0.000000 -0.000000 0.000000 -> xyz=-0.009905 -0.263715 -0.017851 rpy=0.000000 -0.000000 0.000000
- joint joint_RPIN: origin xyz=0.007230 -0.142650 -0.037649 rpy=0.000000 -0.000000 0.000000 -> xyz=0.001692 -0.152650 -0.049495 rpy=0.000000 -0.000000 0.000000
- joint joint_RPSI: origin xyz=-0.100829 -0.002592 0.058275 rpy=0.000000 -0.000000 0.000000 -> xyz=-0.090263 -0.004882 0.058440 rpy=0.000000 -0.000000 0.000000
- joint joint_RSHO: origin xyz=-0.028144 -0.001419 0.165794 rpy=0.000000 -0.000000 0.000000 -> xyz=-0.019136 0.004174 0.174861 rpy=0.000000 -0.000000 0.000000
- joint joint_RTHU: origin xyz=0.006741 -0.114231 0.039600 rpy=0.000000 -0.000000 0.000000 -> xyz=0.005240 -0.097608 0.043099 rpy=0.000000 -0.000000 0.000000
- joint joint_RTOE: origin xyz=0.214550 -0.035325 -0.038104 rpy=0.000000 -0.000000 0.000000 -> xyz=0.216042 -0.033219 -0.041380 rpy=0.000000 -0.000000 0.000000
- joint joint_RWRI: origin xyz=-0.007080 -0.265750 0.017250 rpy=0.000000 -0.000000 0.000000 -> xyz=-0.008906 -0.257846 0.020998 rpy=0.000000 -0.000000 0.000000
- joint joint_T11: origin xyz=-0.134230 0.226914 -0.005502 rpy=0.000000 -0.000000 0.000000 -> xyz=-0.130015 0.214272 0.000267 rpy=0.000000 -0.000000 0.000000
- joint joint_T6: origin xyz=-0.135257 0.214055 0.000164 rpy=0.000000 -0.000000 0.000000 -> xyz=-0.134384 0.198279 0.006296 rpy=0.000000 -0.000000 0.000000
- joint left_ankle_Z: origin xyz=0.000000 -0.417170 0.000000 rpy=0.000000 -0.000000 0.000000 -> xyz=0.000000 -0.434835 0.000000 rpy=0.000000 -0.000000 0.000000
- joint left_clavicle_joint_X: origin xyz=0.000000 0.326014 0.000000 rpy=0.000000 -0.000000 0.000000 -> xyz=0.000000 0.304494 0.000000 rpy=0.000000 -0.000000 0.000000
- joint left_elbow_Z: origin xyz=0.000000 -0.285475 0.000000 rpy=0.000000 -0.000000 0.000000 -> xyz=0.000000 -0.286701 0.000000 rpy=0.000000 -0.000000 0.000000
- joint left_hip_Z: origin xyz=0.025202 -0.090493 -0.088598 rpy=0.000000 -0.000000 0.000000 -> xyz=0.019358 -0.088232 -0.085621 rpy=0.000000 -0.000000 0.000000
- joint left_knee_Z: origin xyz=0.000000 -0.387698 0.000000 rpy=0.000000 -0.000000 0.000000 -> xyz=0.000000 -0.398604 0.000000 rpy=0.000000 -0.000000 0.000000
- joint left_shoulder_Z: origin xyz=0.003712 -0.054580 -0.168501 rpy=0.000000 -0.000000 0.000000 -> xyz=-0.006173 -0.056313 -0.168885 rpy=0.000000 -0.000000 0.000000
- joint left_wrist_Z: origin xyz=0.000000 -0.259369 0.000000 rpy=0.000000 -0.000000 0.000000 -> xyz=0.000000 -0.251410 0.000000 rpy=0.000000 -0.000000 0.000000
- joint middle_cervical_Z: origin xyz=0.000000 0.354247 0.000000 rpy=0.000000 -0.000000 0.000000 -> xyz=0.000000 0.346796 0.000000 rpy=0.000000 -0.000000 0.000000
- joint middle_thoracic_Z: origin xyz=0.000000 0.150702 0.000000 rpy=0.000000 -0.000000 0.000000 -> xyz=0.000000 0.150857 0.000000 rpy=0.000000 -0.000000 0.000000
- joint right_ankle_Z: origin xyz=0.000000 -0.422321 0.000000 rpy=0.000000 -0.000000 0.000000 -> xyz=0.000000 -0.440302 0.000000 rpy=0.000000 -0.000000 0.000000
- joint right_clavicle_joint_X: origin xyz=0.000000 0.326014 0.000000 rpy=0.000000 -0.000000 0.000000 -> xyz=0.000000 0.304494 0.000000 rpy=0.000000 -0.000000 0.000000
- joint right_elbow_Z: origin xyz=0.000000 -0.282755 0.000000 rpy=0.000000 -0.000000 0.000000 -> xyz=0.000000 -0.277150 0.000000 rpy=0.000000 -0.000000 0.000000
- joint right_hip_Z: origin xyz=0.025202 -0.090799 0.088284 rpy=0.000000 -0.000000 0.000000 -> xyz=0.019358 -0.087768 0.086097 rpy=0.000000 -0.000000 0.000000
- joint right_knee_Z: origin xyz=0.000000 -0.391877 0.000000 rpy=0.000000 -0.000000 0.000000 -> xyz=0.000000 -0.406429 0.000000 rpy=0.000000 -0.000000 0.000000
- joint right_shoulder_Z: origin xyz=-0.003712 -0.060044 0.168501 rpy=0.000000 -0.000000 0.000000 -> xyz=0.006173 -0.058608 0.168885 rpy=0.000000 -0.000000 0.000000
- joint right_wrist_Z: origin xyz=0.000000 -0.267516 0.000000 rpy=0.000000 -0.000000 0.000000 -> xyz=0.000000 -0.262101 0.000000 rpy=0.000000 -0.000000 0.000000
