Commit message: rename robot_description topic

File: urdf/human_scaled.urdf (robot description, URDF)
Before this commit: robot human_scaled, 80 links, 79 joints
Joints:
- joint joint_C7: origin xyz=-0.099200 0.343685 0.007565 rpy=0.000000 -0.000000 0.000000 -> xyz=-0.094732 0.363437 0.000272 rpy=0.000000 -0.000000 0.000000
- joint joint_Head: origin xyz=-0.037045 0.265947 -0.003309 rpy=0.000000 -0.000000 0.000000 -> xyz=-0.045813 0.277026 -0.016156 rpy=0.000000 -0.000000 0.000000
- joint joint_L5MHD: origin xyz=0.152476 -0.044943 -0.041387 rpy=0.000000 -0.000000 0.000000 -> xyz=0.160182 -0.042424 -0.039591 rpy=0.000000 -0.000000 0.000000
- joint joint_LANK: origin xyz=-0.004114 -0.437364 -0.030383 rpy=0.000000 -0.000000 0.000000 -> xyz=-0.007232 -0.444898 -0.033953 rpy=0.000000 -0.000000 0.000000
- joint joint_LASI: origin xyz=0.096046 0.000442 -0.119931 rpy=0.000000 -0.000000 0.000000 -> xyz=0.102284 -0.001241 -0.124399 rpy=0.000000 -0.000000 0.000000
- joint joint_LELB: origin xyz=0.020817 -0.278353 -0.022552 rpy=0.000000 -0.000000 0.000000 -> xyz=0.019872 -0.286033 -0.029213 rpy=0.000000 -0.000000 0.000000
- joint joint_LEar: origin xyz=-0.019141 0.141001 -0.077093 rpy=0.000000 -0.000000 0.000000 -> xyz=-0.017107 0.150498 -0.094416 rpy=0.000000 -0.000000 0.000000
- joint joint_LEye: origin xyz=0.100696 0.165863 -0.047471 rpy=0.000000 -0.000000 0.000000 -> xyz=0.081935 0.197090 -0.066894 rpy=0.000000 -0.000000 0.000000
- joint joint_LHEE: origin xyz=-0.064002 -0.041486 0.005135 rpy=0.000000 -0.000000 0.000000 -> xyz=-0.066672 -0.042593 0.004562 rpy=0.000000 -0.000000 0.000000
- joint joint_LKNE: origin xyz=0.018240 -0.400951 -0.055369 rpy=0.000000 -0.000000 0.000000 -> xyz=0.015121 -0.400490 -0.054835 rpy=0.000000 -0.000000 0.000000
- joint joint_LMANK: origin xyz=0.004044 -0.435735 0.035388 rpy=0.000000 -0.000000 0.000000 -> xyz=0.006961 -0.441962 0.036069 rpy=0.000000 -0.000000 0.000000
- joint joint_LMELB: origin xyz=-0.017899 -0.293941 0.052578 rpy=0.000000 -0.000000 0.000000 -> xyz=-0.016917 -0.295805 0.054004 rpy=0.000000 -0.000000 0.000000
- joint joint_LMID: origin xyz=0.000072 -0.121823 -0.000218 rpy=0.000000 -0.000000 0.000000 -> xyz=-0.000075 -0.128615 -0.000133 rpy=0.000000 -0.000000 0.000000
- joint joint_LMKNE: origin xyz=-0.018009 -0.399728 0.053041 rpy=0.000000 -0.000000 0.000000 -> xyz=-0.014666 -0.399625 0.058599 rpy=0.000000 -0.000000 0.000000
- joint joint_LMWRI: origin xyz=-0.008673 -0.255701 0.020159 rpy=0.000000 -0.000000 0.000000 -> xyz=-0.006506 -0.259936 0.022722 rpy=0.000000 -0.000000 0.000000
- joint joint_LPIN: origin xyz=0.008471 -0.144385 0.052178 rpy=0.000000 -0.000000 0.000000 -> xyz=0.013955 -0.128964 0.047523 rpy=0.000000 -0.000000 0.000000
- joint joint_LPSI: origin xyz=-0.085300 -0.004126 -0.056365 rpy=0.000000 -0.000000 0.000000 -> xyz=-0.101837 -0.002786 -0.060705 rpy=0.000000 -0.000000 0.000000
- joint joint_LSHO: origin xyz=-0.038838 0.006150 -0.162456 rpy=0.000000 -0.000000 0.000000 -> xyz=-0.034143 0.007389 -0.172981 rpy=0.000000 -0.000000 0.000000
- joint joint_LTHU: origin xyz=0.004512 -0.091306 -0.055733 rpy=0.000000 -0.000000 0.000000 -> xyz=0.002180 -0.127100 -0.056172 rpy=0.000000 -0.000000 0.000000
- joint joint_LTOE: origin xyz=0.198641 -0.035147 0.023752 rpy=0.000000 -0.000000 0.000000 -> xyz=0.203605 -0.039378 0.025393 rpy=0.000000 -0.000000 0.000000
- joint joint_LWRI: origin xyz=-0.007653 -0.245097 -0.021676 rpy=0.000000 -0.000000 0.000000 -> xyz=-0.006341 -0.258749 -0.024338 rpy=0.000000 -0.000000 0.000000
- joint joint_Nose: origin xyz=0.149182 0.129668 -0.022498 rpy=0.000000 -0.000000 0.000000 -> xyz=0.130070 0.163208 -0.039787 rpy=0.000000 -0.000000 0.000000
- joint joint_R5MHD: origin xyz=0.141127 -0.057036 0.040700 rpy=0.000000 -0.000000 0.000000 -> xyz=0.159887 -0.055583 0.037801 rpy=0.000000 -0.000000 0.000000
- joint joint_RANK: origin xyz=-0.003248 -0.441391 0.031198 rpy=0.000000 -0.000000 0.000000 -> xyz=-0.010131 -0.447277 0.033364 rpy=0.000000 -0.000000 0.000000
- joint joint_RASI: origin xyz=0.091055 0.001004 0.117854 rpy=0.000000 -0.000000 0.000000 -> xyz=0.101042 -0.001397 0.121506 rpy=0.000000 -0.000000 0.000000
- joint joint_RELB: origin xyz=0.024132 -0.267544 0.021595 rpy=0.000000 -0.000000 0.000000 -> xyz=0.026058 -0.271924 0.026577 rpy=0.000000 -0.000000 0.000000
- joint joint_REar: origin xyz=-0.016668 0.144907 0.072865 rpy=0.000000 -0.000000 0.000000 -> xyz=-0.012084 0.155851 0.065578 rpy=0.000000 -0.000000 0.000000
- joint joint_REye: origin xyz=0.098913 0.168377 0.015136 rpy=0.000000 -0.000000 0.000000 -> xyz=0.079463 0.197698 0.002735 rpy=0.000000 -0.000000 0.000000
- joint joint_RHEE: origin xyz=-0.057636 -0.045291 -0.011545 rpy=0.000000 -0.000000 0.000000 -> xyz=-0.072084 -0.050443 -0.007127 rpy=0.000000 -0.000000 0.000000
- joint joint_RKNE: origin xyz=0.008091 -0.408566 0.059432 rpy=0.000000 -0.000000 0.000000 -> xyz=0.010287 -0.411869 0.060971 rpy=0.000000 -0.000000 0.000000
- joint joint_RMANK: origin xyz=0.005676 -0.441949 -0.036535 rpy=0.000000 -0.000000 0.000000 -> xyz=0.009536 -0.442994 -0.037009 rpy=0.000000 -0.000000 0.000000
- joint joint_RMELB: origin xyz=-0.020245 -0.285325 -0.057262 rpy=0.000000 -0.000000 0.000000 -> xyz=-0.020433 -0.289277 -0.058060 rpy=0.000000 -0.000000 0.000000
- joint joint_RMID: origin xyz=0.000499 -0.133794 0.000161 rpy=0.000000 -0.000000 0.000000 -> xyz=0.000080 -0.137609 0.000093 rpy=0.000000 -0.000000 0.000000
- joint joint_RMKNE: origin xyz=-0.022023 -0.407247 -0.053934 rpy=0.000000 -0.000000 0.000000 -> xyz=-0.009995 -0.409755 -0.056347 rpy=0.000000 -0.000000 0.000000
- joint joint_RMWRI: origin xyz=-0.009905 -0.263715 -0.017851 rpy=0.000000 -0.000000 0.000000 -> xyz=-0.008285 -0.270246 -0.024100 rpy=0.000000 -0.000000 0.000000
- joint joint_RPIN: origin xyz=0.001692 -0.152650 -0.049495 rpy=0.000000 -0.000000 0.000000 -> xyz=0.012158 -0.148612 -0.052697 rpy=0.000000 -0.000000 0.000000
- joint joint_RPSI: origin xyz=-0.090263 -0.004882 0.058440 rpy=0.000000 -0.000000 0.000000 -> xyz=-0.098164 -0.004014 0.059074 rpy=0.000000 -0.000000 0.000000
- joint joint_RSHO: origin xyz=-0.019136 0.004174 0.174861 rpy=0.000000 -0.000000 0.000000 -> xyz=-0.019471 -0.003183 0.173189 rpy=0.000000 -0.000000 0.000000
- joint joint_RTHU: origin xyz=0.005240 -0.097608 0.043099 rpy=0.000000 -0.000000 0.000000 -> xyz=0.007281 -0.113641 0.056225 rpy=0.000000 -0.000000 0.000000
- joint joint_RTOE: origin xyz=0.216042 -0.033219 -0.041380 rpy=0.000000 -0.000000 0.000000 -> xyz=0.237660 -0.040074 -0.037635 rpy=0.000000 -0.000000 0.000000
- joint joint_RWRI: origin xyz=-0.008906 -0.257846 0.020998 rpy=0.000000 -0.000000 0.000000 -> xyz=-0.006814 -0.273341 0.023422 rpy=0.000000 -0.000000 0.000000
- joint joint_T11: origin xyz=-0.130015 0.214272 0.000267 rpy=0.000000 -0.000000 0.000000 -> xyz=-0.146801 0.226085 -0.003078 rpy=0.000000 -0.000000 0.000000
- joint joint_T6: origin xyz=-0.134384 0.198279 0.006296 rpy=0.000000 -0.000000 0.000000 -> xyz=-0.148961 0.214853 0.000566 rpy=0.000000 -0.000000 0.000000
- joint left_ankle_Z: origin xyz=0.000000 -0.434835 0.000000 rpy=0.000000 -0.000000 0.000000 -> xyz=0.000000 -0.441434 0.000000 rpy=0.000000 -0.000000 0.000000
- joint left_clavicle_joint_X: origin xyz=0.000000 0.304494 0.000000 rpy=0.000000 -0.000000 0.000000 -> xyz=0.000000 0.326640 0.000000 rpy=0.000000 -0.000000 0.000000
- joint left_elbow_Z: origin xyz=0.000000 -0.286701 0.000000 rpy=0.000000 -0.000000 0.000000 -> xyz=0.000000 -0.291479 0.000000 rpy=0.000000 -0.000000 0.000000
- joint left_hip_Z: origin xyz=0.019358 -0.088232 -0.085621 rpy=0.000000 -0.000000 0.000000 -> xyz=0.027065 -0.091276 -0.088475 rpy=0.000000 -0.000000 0.000000
- joint left_knee_Z: origin xyz=0.000000 -0.398604 0.000000 rpy=0.000000 -0.000000 0.000000 -> xyz=0.000000 -0.398047 0.000000 rpy=0.000000 -0.000000 0.000000
- joint left_shoulder_Z: origin xyz=-0.006173 -0.056313 -0.168885 rpy=0.000000 -0.000000 0.000000 -> xyz=-0.005127 -0.053255 -0.173145 rpy=0.000000 -0.000000 0.000000
- joint left_wrist_Z: origin xyz=0.000000 -0.251410 0.000000 rpy=0.000000 -0.000000 0.000000 -> xyz=0.000000 -0.259826 0.000000 rpy=0.000000 -0.000000 0.000000
- joint middle_cervical_Z: origin xyz=0.000000 0.346796 0.000000 rpy=0.000000 -0.000000 0.000000 -> xyz=0.000000 0.353783 0.000000 rpy=0.000000 -0.000000 0.000000
- joint middle_thoracic_Z: origin xyz=0.000000 0.150857 0.000000 rpy=0.000000 -0.000000 0.000000 -> xyz=0.000000 0.151074 0.000000 rpy=0.000000 -0.000000 0.000000
- joint right_ankle_Z: origin xyz=0.000000 -0.440302 0.000000 rpy=0.000000 -0.000000 0.000000 -> xyz=0.000000 -0.442597 0.000000 rpy=0.000000 -0.000000 0.000000
- joint right_clavicle_joint_X: origin xyz=0.000000 0.304494 0.000000 rpy=0.000000 -0.000000 0.000000 -> xyz=0.000000 0.326640 0.000000 rpy=0.000000 -0.000000 0.000000
- joint right_elbow_Z: origin xyz=0.000000 -0.277150 0.000000 rpy=0.000000 -0.000000 0.000000 -> xyz=0.000000 -0.281571 0.000000 rpy=0.000000 -0.000000 0.000000
- joint right_hip_Z: origin xyz=0.019358 -0.087768 0.086097 rpy=0.000000 -0.000000 0.000000 -> xyz=0.027065 -0.090695 0.089070 rpy=0.000000 -0.000000 0.000000
- joint right_knee_Z: origin xyz=0.000000 -0.406429 0.000000 rpy=0.000000 -0.000000 0.000000 -> xyz=0.000000 -0.408248 0.000000 rpy=0.000000 -0.000000 0.000000
- joint right_shoulder_Z: origin xyz=0.006173 -0.058608 0.168885 rpy=0.000000 -0.000000 0.000000 -> xyz=0.005127 -0.064598 0.173145 rpy=0.000000 -0.000000 0.000000
- joint right_wrist_Z: origin xyz=0.000000 -0.262101 0.000000 rpy=0.000000 -0.000000 0.000000 -> xyz=0.000000 -0.272273 0.000000 rpy=0.000000 -0.000000 0.000000

Commit message: add capsules for left arm, thorax and head

File: urdf/human_scaled.urdf (robot description, URDF)
Before this commit: robot human_scaled, 80 links, 79 joints
Joints:
- joint joint_C7: origin xyz=-0.094732 0.363437 0.000272 rpy=0.000000 -0.000000 0.000000 -> xyz=-0.111923 0.374361 0.005497 rpy=0.000000 -0.000000 0.000000
- joint joint_Head: origin xyz=-0.045813 0.277026 -0.016156 rpy=0.000000 -0.000000 0.000000 -> xyz=-0.025305 0.280497 0.019934 rpy=0.000000 -0.000000 0.000000
- joint joint_L5MHD: origin xyz=0.160182 -0.042424 -0.039591 rpy=0.000000 -0.000000 0.000000 -> xyz=0.134114 -0.050876 -0.053920 rpy=0.000000 -0.000000 0.000000
- joint joint_LANK: origin xyz=-0.007232 -0.444898 -0.033953 rpy=0.000000 -0.000000 0.000000 -> xyz=-0.013731 -0.443231 -0.039504 rpy=0.000000 -0.000000 0.000000
- joint joint_LASI: origin xyz=0.102284 -0.001241 -0.124399 rpy=0.000000 -0.000000 0.000000 -> xyz=0.068360 -0.013725 -0.127581 rpy=0.000000 -0.000000 0.000000
- joint joint_LELB: origin xyz=0.019872 -0.286033 -0.029213 rpy=0.000000 -0.000000 0.000000 -> xyz=0.015725 -0.277010 -0.017679 rpy=0.000000 -0.000000 0.000000
- joint joint_LEar: origin xyz=-0.017107 0.150498 -0.094416 rpy=0.000000 -0.000000 0.000000 -> xyz=-0.018169 0.150982 -0.065592 rpy=0.000000 -0.000000 0.000000
- joint joint_LEye: origin xyz=0.081935 0.197090 -0.066894 rpy=0.000000 -0.000000 0.000000 -> xyz=0.120538 0.153713 -0.003514 rpy=0.000000 -0.000000 0.000000
- joint joint_LHEE: origin xyz=-0.066672 -0.042593 0.004562 rpy=0.000000 -0.000000 0.000000 -> xyz=-0.070497 -0.041123 -0.002756 rpy=0.000000 -0.000000 0.000000
- joint joint_LKNE: origin xyz=0.015121 -0.400490 -0.054835 rpy=0.000000 -0.000000 0.000000 -> xyz=0.011749 -0.372980 -0.046821 rpy=0.000000 -0.000000 0.000000
- joint joint_LMANK: origin xyz=0.006961 -0.441962 0.036069 rpy=0.000000 -0.000000 0.000000 -> xyz=0.013752 -0.433247 0.036791 rpy=0.000000 -0.000000 0.000000
- joint joint_LMELB: origin xyz=-0.016917 -0.295805 0.054004 rpy=0.000000 -0.000000 0.000000 -> xyz=-0.013417 -0.287073 0.045780 rpy=0.000000 -0.000000 0.000000
- joint joint_LMID: origin xyz=-0.000075 -0.128615 -0.000133 rpy=0.000000 -0.000000 0.000000 -> xyz=0.000158 -0.118830 -0.000086 rpy=0.000000 -0.000000 0.000000
- joint joint_LMKNE: origin xyz=-0.014666 -0.399625 0.058599 rpy=0.000000 -0.000000 0.000000 -> xyz=-0.010001 -0.370675 0.072922 rpy=0.000000 -0.000000 0.000000
- joint joint_LMWRI: origin xyz=-0.006506 -0.259936 0.022722 rpy=0.000000 -0.000000 0.000000 -> xyz=-0.008199 -0.246444 0.015818 rpy=0.000000 -0.000000 0.000000
- joint joint_LPIN: origin xyz=0.013955 -0.128964 0.047523 rpy=0.000000 -0.000000 0.000000 -> xyz=0.005591 -0.133267 0.031496 rpy=0.000000 -0.000000 0.000000
- joint joint_LPSI: origin xyz=-0.101837 -0.002786 -0.060705 rpy=0.000000 -0.000000 0.000000 -> xyz=-0.078210 0.002657 -0.056720 rpy=0.000000 -0.000000 0.000000
- joint joint_LSHO: origin xyz=-0.034143 0.007389 -0.172981 rpy=0.000000 -0.000000 0.000000 -> xyz=-0.031782 0.008956 -0.166478 rpy=0.000000 -0.000000 0.000000
- joint joint_LTHU: origin xyz=0.002180 -0.127100 -0.056172 rpy=0.000000 -0.000000 0.000000 -> xyz=0.006212 -0.092085 -0.033361 rpy=0.000000 -0.000000 0.000000
- joint joint_LTOE: origin xyz=0.203605 -0.039378 0.025393 rpy=0.000000 -0.000000 0.000000 -> xyz=0.205957 -0.027467 0.024858 rpy=0.000000 -0.000000 0.000000
- joint joint_LWRI: origin xyz=-0.006341 -0.258749 -0.024338 rpy=0.000000 -0.000000 0.000000 -> xyz=-0.007147 -0.235756 -0.014928 rpy=0.000000 -0.000000 0.000000
- joint joint_Nose: origin xyz=0.130070 0.163208 -0.039787 rpy=0.000000 -0.000000 0.000000 -> xyz=0.168114 0.105911 0.030550 rpy=0.000000 -0.000000 0.000000
- joint joint_R5MHD: origin xyz=0.159887 -0.055583 0.037801 rpy=0.000000 -0.000000 0.000000 -> xyz=0.122945 -0.017119 0.031094 rpy=0.000000 -0.000000 0.000000
- joint joint_RANK: origin xyz=-0.010131 -0.447277 0.033364 rpy=0.000000 -0.000000 0.000000 -> xyz=0.026776 -0.412372 -0.006134 rpy=0.000000 -0.000000 0.000000
- joint joint_RASI: origin xyz=0.101042 -0.001397 0.121506 rpy=0.000000 -0.000000 0.000000 -> xyz=0.072973 -0.004670 0.137746 rpy=0.000000 -0.000000 0.000000
- joint joint_RELB: origin xyz=0.026058 -0.271924 0.026577 rpy=0.000000 -0.000000 0.000000 -> xyz=0.018990 -0.280749 0.022614 rpy=0.000000 -0.000000 0.000000
- joint joint_REar: origin xyz=-0.012084 0.155851 0.065578 rpy=0.000000 -0.000000 0.000000 -> xyz=-0.023065 0.138062 0.084845 rpy=0.000000 -0.000000 0.000000
- joint joint_REye: origin xyz=0.079463 0.197698 0.002735 rpy=0.000000 -0.000000 0.000000 -> xyz=0.123623 0.147197 0.062523 rpy=0.000000 -0.000000 0.000000
- joint joint_RHEE: origin xyz=-0.072084 -0.050443 -0.007127 rpy=0.000000 -0.000000 0.000000 -> xyz=0.010354 0.000286 -0.061308 rpy=0.000000 -0.000000 0.000000
- joint joint_RKNE: origin xyz=0.010287 -0.411869 0.060971 rpy=0.000000 -0.000000 0.000000 -> xyz=0.019239 -0.394820 0.042566 rpy=0.000000 -0.000000 0.000000
- joint joint_RMANK: origin xyz=0.009536 -0.442994 -0.037009 rpy=0.000000 -0.000000 0.000000 -> xyz=-0.019286 -0.443148 -0.058842 rpy=0.000000 -0.000000 0.000000
- joint joint_RMELB: origin xyz=-0.020433 -0.289277 -0.058060 rpy=0.000000 -0.000000 0.000000 -> xyz=-0.018748 -0.292968 -0.047333 rpy=0.000000 -0.000000 0.000000
- joint joint_RMID: origin xyz=0.000080 -0.137609 0.000093 rpy=0.000000 -0.000000 0.000000 -> xyz=0.000367 -0.137894 0.000150 rpy=0.000000 -0.000000 0.000000
- joint joint_RMKNE: origin xyz=-0.009995 -0.409755 -0.056347 rpy=0.000000 -0.000000 0.000000 -> xyz=-0.019234 -0.392180 -0.081665 rpy=0.000000 -0.000000 0.000000
- joint joint_RMWRI: origin xyz=-0.008285 -0.270246 -0.024100 rpy=0.000000 -0.000000 0.000000 -> xyz=-0.007154 -0.264752 -0.017388 rpy=0.000000 -0.000000 0.000000
- joint joint_RPIN: origin xyz=0.012158 -0.148612 -0.052697 rpy=0.000000 -0.000000 0.000000 -> xyz=0.002559 -0.159945 -0.047535 rpy=0.000000 -0.000000 0.000000
- joint joint_RPSI: origin xyz=-0.098164 -0.004014 0.059074 rpy=0.000000 -0.000000 0.000000 -> xyz=-0.072023 0.004415 0.064792 rpy=0.000000 -0.000000 0.000000
- joint joint_RSHO: origin xyz=-0.019471 -0.003183 0.173189 rpy=0.000000 -0.000000 0.000000 -> xyz=-0.027063 0.000745 0.177333 rpy=0.000000 -0.000000 0.000000
- joint joint_RTHU: origin xyz=0.007281 -0.113641 0.056225 rpy=0.000000 -0.000000 0.000000 -> xyz=0.006278 -0.100421 0.039918 rpy=0.000000 -0.000000 0.000000
- joint joint_RTOE: origin xyz=0.237660 -0.040074 -0.037635 rpy=0.000000 -0.000000 0.000000 -> xyz=0.138472 -0.041739 -0.039254 rpy=0.000000 -0.000000 0.000000
- joint joint_RWRI: origin xyz=-0.006814 -0.273341 0.023422 rpy=0.000000 -0.000000 0.000000 -> xyz=-0.006259 -0.257874 0.019761 rpy=0.000000 -0.000000 0.000000
- joint joint_T11: origin xyz=-0.146801 0.226085 -0.003078 rpy=0.000000 -0.000000 0.000000 -> xyz=-0.130494 0.222348 -0.001312 rpy=0.000000 -0.000000 0.000000
- joint joint_T6: origin xyz=-0.148961 0.214853 0.000566 rpy=0.000000 -0.000000 0.000000 -> xyz=-0.131836 0.225908 0.000555 rpy=0.000000 -0.000000 0.000000
- joint left_ankle_Z: origin xyz=0.000000 -0.441434 0.000000 rpy=0.000000 -0.000000 0.000000 -> xyz=0.000000 -0.436487 0.000000 rpy=0.000000 -0.000000 0.000000
- joint left_clavicle_joint_X: origin xyz=0.000000 0.326640 0.000000 rpy=0.000000 -0.000000 0.000000 -> xyz=0.000000 0.329314 0.000000 rpy=0.000000 -0.000000 0.000000
- joint left_elbow_Z: origin xyz=0.000000 -0.291479 0.000000 rpy=0.000000 -0.000000 0.000000 -> xyz=0.000000 -0.282811 0.000000 rpy=0.000000 -0.000000 0.000000
- joint left_hip_Z: origin xyz=0.027065 -0.091276 -0.088475 rpy=0.000000 -0.000000 0.000000 -> xyz=-0.006486 -0.098743 -0.095338 rpy=0.000000 -0.000000 0.000000
- joint left_knee_Z: origin xyz=0.000000 -0.398047 0.000000 rpy=0.000000 -0.000000 0.000000 -> xyz=0.000000 -0.369602 0.000000 rpy=0.000000 -0.000000 0.000000
- joint left_shoulder_Z: origin xyz=-0.005127 -0.053255 -0.173145 rpy=0.000000 -0.000000 0.000000 -> xyz=-0.001260 -0.050254 -0.171838 rpy=0.000000 -0.000000 0.000000
- joint left_wrist_Z: origin xyz=0.000000 -0.259826 0.000000 rpy=0.000000 -0.000000 0.000000 -> xyz=0.000000 -0.242503 0.000000 rpy=0.000000 -0.000000 0.000000
- joint middle_cervical_Z: origin xyz=0.000000 0.353783 0.000000 rpy=0.000000 -0.000000 0.000000 -> xyz=0.000000 0.375732 0.000000 rpy=0.000000 -0.000000 0.000000
- joint middle_thoracic_Z: origin xyz=0.000000 0.151074 0.000000 rpy=0.000000 -0.000000 0.000000 -> xyz=0.000000 0.147432 0.000000 rpy=0.000000 -0.000000 0.000000
- joint right_ankle_Z: origin xyz=0.000000 -0.442597 0.000000 rpy=0.000000 -0.000000 0.000000 -> xyz=0.000000 -0.429759 0.000000 rpy=0.000000 -0.000000 0.000000
- joint right_clavicle_joint_X: origin xyz=0.000000 0.326640 0.000000 rpy=0.000000 -0.000000 0.000000 -> xyz=0.000000 0.329314 0.000000 rpy=0.000000 -0.000000 0.000000
- joint right_elbow_Z: origin xyz=0.000000 -0.281571 0.000000 rpy=0.000000 -0.000000 0.000000 -> xyz=0.000000 -0.286027 0.000000 rpy=0.000000 -0.000000 0.000000
- joint right_hip_Z: origin xyz=0.027065 -0.090695 0.089070 rpy=0.000000 -0.000000 0.000000 -> xyz=-0.006486 -0.097740 0.096366 rpy=0.000000 -0.000000 0.000000
- joint right_knee_Z: origin xyz=0.000000 -0.408248 0.000000 rpy=0.000000 -0.000000 0.000000 -> xyz=0.000000 -0.395293 0.000000 rpy=0.000000 -0.000000 0.000000
- joint right_shoulder_Z: origin xyz=0.005127 -0.064598 0.173145 rpy=0.000000 -0.000000 0.000000 -> xyz=0.001260 -0.066733 0.171838 rpy=0.000000 -0.000000 0.000000
- joint right_wrist_Z: origin xyz=0.000000 -0.272273 0.000000 rpy=0.000000 -0.000000 0.000000 -> xyz=0.000000 -0.261213 0.000000 rpy=0.000000 -0.000000 0.000000
