Commit message: rework for new cosmik

File: urdf/human_scaled.urdf (robot description, URDF)
Before this commit: robot human_scaled, 80 links, 79 joints
Links:
- link middle_abdomen: geometry visual mesh filename=package://rtcosmik_ros/meshes/abdomen_mesh.STL scale=0.005100 0.005100 0.005100
- link middle_pelvis: geometry visual mesh filename=package://rtcosmik_ros/meshes/pelvis_mesh.STL scale=0.006464 0.005930 0.005930
- link middle_thorax: geometry visual mesh filename=package://rtcosmik_ros/meshes/torso_mesh.STL scale=0.005815 0.009144 0.005815
Joints:
- joint joint_C7: origin xyz=-0.111923 0.374361 0.005497 rpy=0.000000 -0.000000 0.000000 -> xyz=-0.080403 0.304940 -0.001789 rpy=0.000000 -0.000000 0.000000
- joint joint_Head: origin xyz=-0.025305 0.280497 0.019934 rpy=0.000000 -0.000000 0.000000 -> xyz=-0.042938 0.258525 -0.005349 rpy=0.000000 -0.000000 0.000000
- joint joint_L5MHD: origin xyz=0.134114 -0.050876 -0.053920 rpy=0.000000 -0.000000 0.000000 -> xyz=0.138644 -0.035999 -0.041912 rpy=0.000000 -0.000000 0.000000
- joint joint_LANK: origin xyz=-0.013731 -0.443231 -0.039504 rpy=0.000000 -0.000000 0.000000 -> xyz=-0.003708 -0.462206 -0.033679 rpy=0.000000 -0.000000 0.000000
- joint joint_LASI: origin xyz=0.068360 -0.013725 -0.127581 rpy=0.000000 -0.000000 0.000000 -> xyz=0.084222 -0.002758 -0.115229 rpy=0.000000 -0.000000 0.000000
- joint joint_LELB: origin xyz=0.015725 -0.277010 -0.017679 rpy=0.000000 -0.000000 0.000000 -> xyz=0.013404 -0.278677 -0.018009 rpy=0.000000 -0.000000 0.000000
- joint joint_LEar: origin xyz=-0.018169 0.150982 -0.065592 rpy=0.000000 -0.000000 0.000000 -> xyz=-0.012661 0.127764 -0.077262 rpy=0.000000 -0.000000 0.000000
- joint joint_LEye: origin xyz=0.120538 0.153713 -0.003514 rpy=0.000000 -0.000000 0.000000 -> xyz=0.075322 0.161414 -0.036531 rpy=0.000000 -0.000000 0.000000
- joint joint_LHEE: origin xyz=-0.070497 -0.041123 -0.002756 rpy=0.000000 -0.000000 0.000000 -> xyz=-0.054828 -0.033255 0.000761 rpy=0.000000 -0.000000 0.000000
- joint joint_LKNE: origin xyz=0.011749 -0.372980 -0.046821 rpy=0.000000 -0.000000 0.000000 -> xyz=0.009129 -0.395153 -0.046892 rpy=0.000000 -0.000000 0.000000
- joint joint_LMANK: origin xyz=0.013752 -0.433247 0.036791 rpy=0.000000 -0.000000 0.000000 -> xyz=0.003952 -0.457384 0.031801 rpy=0.000000 -0.000000 0.000000
- joint joint_LMELB: origin xyz=-0.013417 -0.287073 0.045780 rpy=0.000000 -0.000000 0.000000 -> xyz=-0.012587 -0.286336 0.056077 rpy=0.000000 -0.000000 0.000000
- joint joint_LMID: origin xyz=0.000158 -0.118830 -0.000086 rpy=0.000000 -0.000000 0.000000 -> xyz=-0.001265 -0.127797 -0.002368 rpy=0.000000 -0.000000 0.000000
- joint joint_LMKNE: origin xyz=-0.010001 -0.370675 0.072922 rpy=0.000000 -0.000000 0.000000 -> xyz=-0.009133 -0.388279 0.063135 rpy=0.000000 -0.000000 0.000000
- joint joint_LMWRI: origin xyz=-0.008199 -0.246444 0.015818 rpy=0.000000 -0.000000 0.000000 -> xyz=-0.016401 -0.246420 0.009986 rpy=0.000000 -0.000000 0.000000
- joint joint_LPIN: origin xyz=0.005591 -0.133267 0.031496 rpy=0.000000 -0.000000 0.000000 -> xyz=0.004875 -0.144521 0.024714 rpy=0.000000 -0.000000 0.000000
- joint joint_LPSI: origin xyz=-0.078210 0.002657 -0.056720 rpy=0.000000 -0.000000 0.000000 -> xyz=-0.084374 0.002051 -0.058808 rpy=0.000000 -0.000000 0.000000
- joint joint_LSHO: origin xyz=-0.031782 0.008956 -0.166478 rpy=0.000000 -0.000000 0.000000 -> xyz=-0.011227 0.004744 -0.156694 rpy=0.000000 -0.000000 0.000000
- joint joint_LTHU: origin xyz=0.006212 -0.092085 -0.033361 rpy=0.000000 -0.000000 0.000000 -> xyz=0.017502 -0.101302 -0.042385 rpy=0.000000 -0.000000 0.000000
- joint joint_LTOE: origin xyz=0.205957 -0.027467 0.024858 rpy=0.000000 -0.000000 0.000000 -> xyz=0.183317 -0.030757 0.027229 rpy=0.000000 -0.000000 0.000000
- joint joint_LWRI: origin xyz=-0.007147 -0.235756 -0.014928 rpy=0.000000 -0.000000 0.000000 -> xyz=-0.004162 -0.241738 -0.021819 rpy=0.000000 -0.000000 0.000000
- joint joint_Nose: origin xyz=0.168114 0.105911 0.030550 rpy=0.000000 -0.000000 0.000000 -> xyz=0.117305 0.116548 -0.003687 rpy=0.000000 -0.000000 0.000000
- joint joint_R5MHD: origin xyz=0.122945 -0.017119 0.031094 rpy=0.000000 -0.000000 0.000000 -> xyz=0.131005 -0.052868 0.036635 rpy=0.000000 -0.000000 0.000000
- joint joint_RANK: origin xyz=0.026776 -0.412372 -0.006134 rpy=0.000000 -0.000000 0.000000 -> xyz=-0.003593 -0.453700 0.030322 rpy=0.000000 -0.000000 0.000000
- joint joint_RASI: origin xyz=0.072973 -0.004670 0.137746 rpy=0.000000 -0.000000 0.000000 -> xyz=0.084514 -0.003155 0.114142 rpy=0.000000 -0.000000 0.000000
- joint joint_RELB: origin xyz=0.018990 -0.280749 0.022614 rpy=0.000000 -0.000000 0.000000 -> xyz=0.012643 -0.274683 0.017820 rpy=0.000000 -0.000000 0.000000
- joint joint_REar: origin xyz=-0.023065 0.138062 0.084845 rpy=0.000000 -0.000000 0.000000 -> xyz=-0.010699 0.125607 0.066083 rpy=0.000000 -0.000000 0.000000
- joint joint_REye: origin xyz=0.123623 0.147197 0.062523 rpy=0.000000 -0.000000 0.000000 -> xyz=0.076730 0.160508 0.026633 rpy=0.000000 -0.000000 0.000000
- joint joint_RHEE: origin xyz=0.010354 0.000286 -0.061308 rpy=0.000000 -0.000000 0.000000 -> xyz=-0.053447 -0.046394 -0.008728 rpy=0.000000 -0.000000 0.000000
- joint joint_RKNE: origin xyz=0.019239 -0.394820 0.042566 rpy=0.000000 -0.000000 0.000000 -> xyz=0.011967 -0.399554 0.052019 rpy=0.000000 -0.000000 0.000000
- joint joint_RMANK: origin xyz=-0.019286 -0.443148 -0.058842 rpy=0.000000 -0.000000 0.000000 -> xyz=0.003366 -0.453382 -0.031911 rpy=0.000000 -0.000000 0.000000
- joint joint_RMELB: origin xyz=-0.018748 -0.292968 -0.047333 rpy=0.000000 -0.000000 0.000000 -> xyz=-0.011456 -0.286480 -0.051546 rpy=0.000000 -0.000000 0.000000
- joint joint_RMID: origin xyz=0.000367 -0.137894 0.000150 rpy=0.000000 -0.000000 0.000000 -> xyz=-0.000233 -0.128281 0.000751 rpy=0.000000 -0.000000 0.000000
- joint joint_RMKNE: origin xyz=-0.019234 -0.392180 -0.081665 rpy=0.000000 -0.000000 0.000000 -> xyz=-0.010461 -0.398982 -0.057720 rpy=0.000000 -0.000000 0.000000
- joint joint_RMWRI: origin xyz=-0.007154 -0.264752 -0.017388 rpy=0.000000 -0.000000 0.000000 -> xyz=-0.013745 -0.245145 -0.011280 rpy=0.000000 -0.000000 0.000000
- joint joint_RPIN: origin xyz=0.002559 -0.159945 -0.047535 rpy=0.000000 -0.000000 0.000000 -> xyz=-0.000626 -0.147241 -0.031849 rpy=0.000000 -0.000000 0.000000
- joint joint_RPSI: origin xyz=-0.072023 0.004415 0.064792 rpy=0.000000 -0.000000 0.000000 -> xyz=-0.084832 -0.000319 0.055091 rpy=0.000000 -0.000000 0.000000
- joint joint_RSHO: origin xyz=-0.027063 0.000745 0.177333 rpy=0.000000 -0.000000 0.000000 -> xyz=-0.017031 -0.005065 0.152077 rpy=0.000000 -0.000000 0.000000
- joint joint_RTHU: origin xyz=0.006278 -0.100421 0.039918 rpy=0.000000 -0.000000 0.000000 -> xyz=0.017843 -0.094398 0.044588 rpy=0.000000 -0.000000 0.000000
- joint joint_RTOE: origin xyz=0.138472 -0.041739 -0.039254 rpy=0.000000 -0.000000 0.000000 -> xyz=0.175883 -0.039904 -0.033033 rpy=0.000000 -0.000000 0.000000
- joint joint_RWRI: origin xyz=-0.006259 -0.257874 0.019761 rpy=0.000000 -0.000000 0.000000 -> xyz=-0.004111 -0.242283 0.021845 rpy=0.000000 -0.000000 0.000000
- joint joint_T11: origin xyz=-0.130494 0.222348 -0.001312 rpy=0.000000 -0.000000 0.000000 -> xyz=-0.099289 0.206912 0.000960 rpy=0.000000 -0.000000 0.000000
- joint joint_T6: origin xyz=-0.131836 0.225908 0.000555 rpy=0.000000 -0.000000 0.000000 -> xyz=-0.107234 0.176306 -0.003218 rpy=0.000000 -0.000000 0.000000
- joint left_ankle_Z: origin xyz=0.000000 -0.436487 0.000000 rpy=0.000000 -0.000000 0.000000 -> xyz=0.000000 -0.459255 0.000000 rpy=0.000000 -0.000000 0.000000
- joint left_clavicle_joint_X: origin xyz=0.000000 0.329314 0.000000 rpy=0.000000 -0.000000 0.000000 -> xyz=0.000000 0.287346 0.000000 rpy=0.000000 -0.000000 0.000000
- joint left_elbow_Z: origin xyz=0.000000 -0.282811 0.000000 rpy=0.000000 -0.000000 0.000000 -> xyz=0.000000 -0.281772 0.000000 rpy=0.000000 -0.000000 0.000000
- joint left_hip_Z: origin xyz=-0.006486 -0.098743 -0.095338 rpy=0.000000 -0.000000 0.000000 -> xyz=0.015698 -0.085393 -0.082261 rpy=0.000000 -0.000000 0.000000
- joint left_knee_Z: origin xyz=0.000000 -0.369602 0.000000 rpy=0.000000 -0.000000 0.000000 -> xyz=0.000000 -0.391086 0.000000 rpy=0.000000 -0.000000 0.000000
- joint left_shoulder_Z: origin xyz=-0.001260 -0.050254 -0.171838 rpy=0.000000 -0.000000 0.000000 -> xyz=0.004617 -0.048239 -0.154356 rpy=0.000000 -0.000000 0.000000
- joint left_wrist_Z: origin xyz=0.000000 -0.242503 0.000000 rpy=0.000000 -0.000000 0.000000 -> xyz=0.000000 -0.245200 0.000000 rpy=0.000000 -0.000000 0.000000
- joint middle_cervical_Z: origin xyz=0.000000 0.375732 0.000000 rpy=0.000000 -0.000000 0.000000 -> xyz=0.000000 0.316179 0.000000 rpy=0.000000 -0.000000 0.000000
- joint middle_thoracic_Z: origin xyz=0.000000 0.147432 0.000000 rpy=0.000000 -0.000000 0.000000 -> xyz=0.000000 0.149427 0.000000 rpy=0.000000 -0.000000 0.000000
- joint right_ankle_Z: origin xyz=0.000000 -0.429759 0.000000 rpy=0.000000 -0.000000 0.000000 -> xyz=0.000000 -0.452413 0.000000 rpy=0.000000 -0.000000 0.000000
- joint right_clavicle_joint_X: origin xyz=0.000000 0.329314 0.000000 rpy=0.000000 -0.000000 0.000000 -> xyz=0.000000 0.287346 0.000000 rpy=0.000000 -0.000000 0.000000
- joint right_elbow_Z: origin xyz=0.000000 -0.286027 0.000000 rpy=0.000000 -0.000000 0.000000 -> xyz=0.000000 -0.279813 0.000000 rpy=0.000000 -0.000000 0.000000
- joint right_hip_Z: origin xyz=-0.006486 -0.097740 0.096366 rpy=0.000000 -0.000000 0.000000 -> xyz=0.015698 -0.084338 0.083342 rpy=0.000000 -0.000000 0.000000
- joint right_knee_Z: origin xyz=0.000000 -0.395293 0.000000 rpy=0.000000 -0.000000 0.000000 -> xyz=0.000000 -0.398015 0.000000 rpy=0.000000 -0.000000 0.000000
- joint right_shoulder_Z: origin xyz=0.001260 -0.066733 0.171838 rpy=0.000000 -0.000000 0.000000 -> xyz=-0.004617 -0.056811 0.154356 rpy=0.000000 -0.000000 0.000000
- joint right_wrist_Z: origin xyz=0.000000 -0.261213 0.000000 rpy=0.000000 -0.000000 0.000000 -> xyz=0.000000 -0.244295 0.000000 rpy=0.000000 -0.000000 0.000000

Commit message: adapt color saturation

File: urdf/human_scaled.urdf (robot description, URDF)
Before this commit: robot human_scaled, 80 links, 79 joints
Links:
- link left_foot: mass 0.89 -> 0.6; geometry visual mesh filename=package://rtcosmik_ros/meshes/foot_mesh.STL scale=0.006100 0.006100 0.006100
- link left_hand: mass 0.44 -> 0.3; geometry visual mesh filename=package://rtcosmik_ros/meshes/hand_mesh.STL scale=0.005500 0.005500 0.005500
- link left_lowerarm: mass 1.26 -> 0.85; geometry visual mesh filename=package://rtcosmik_ros/meshes/elbow_mesh.STL scale=0.005000 0.005000 0.005000; visual mesh filename=package://rtcosmik_ros/meshes/lowerarm_mesh.STL scale=0.005800 0.005800 0.005800
- link left_lowerleg: mass 3.55 -> 2.4; geometry visual mesh filename=package://rtcosmik_ros/meshes/knee_mesh.STL scale=0.005100 0.005100 0.005100; visual mesh filename=package://rtcosmik_ros/meshes/lowerleg_mesh.STL scale=0.005700 0.006000 0.006400
- link left_upperarm: mass 1.78 -> 1.2; geometry visual mesh filename=package://rtcosmik_ros/meshes/shoulder_mesh.STL scale=0.003600 0.003600 0.003600; visual mesh filename=package://rtcosmik_ros/meshes/upperarm_mesh.STL scale=0.005700 0.005500 0.006300
- link left_upperleg: mass 9.1 -> 6.15; geometry visual mesh filename=package://rtcosmik_ros/meshes/upperleg_mesh.STL scale=0.005600 0.005800 0.006300
- link middle_abdomen: mass 12.08 -> 8.16; geometry visual mesh filename=package://rtcosmik_ros/meshes/abdomen_mesh.STL scale=0.004600 0.004600 0.004600
- link middle_head: mass 4.96 -> 3.35; geometry visual mesh filename=package://rtcosmik_ros/meshes/head_mesh.STL scale=0.005100 0.005100 0.005100; visual mesh filename=package://rtcosmik_ros/meshes/neck_mesh.STL scale=0.004500 0.004500 0.004500
- link middle_pelvis: mass 10.51 -> 7.1; geometry visual mesh filename=package://rtcosmik_ros/meshes/pelvis_mesh.STL scale=0.005857 0.005373 0.005373
- link middle_thorax: mass 11.81 -> 7.98; geometry visual mesh filename=package://rtcosmik_ros/meshes/torso_mesh.STL scale=0.005269 0.008285 0.005269
- link right_foot: mass 0.89 -> 0.6; geometry visual mesh filename=package://rtcosmik_ros/meshes/foot_mesh.STL scale=0.006100 0.006100 0.006100
- link right_hand: mass 0.44 -> 0.3; geometry visual mesh filename=package://rtcosmik_ros/meshes/hand_mesh.STL scale=0.005500 0.005500 0.005500
- link right_lowerarm: mass 1.26 -> 0.85; geometry visual mesh filename=package://rtcosmik_ros/meshes/elbow_mesh.STL scale=0.005000 0.005000 0.005000; visual mesh filename=package://rtcosmik_ros/meshes/lowerarm_mesh.STL scale=0.005800 0.005800 0.005800
- link right_lowerleg: mass 3.55 -> 2.4; geometry visual mesh filename=package://rtcosmik_ros/meshes/knee_mesh.STL scale=0.005100 0.005100 0.005100; visual mesh filename=package://rtcosmik_ros/meshes/lowerleg_mesh.STL scale=0.005700 0.006000 0.006400
- link right_upperarm: mass 1.78 -> 1.2; geometry visual mesh filename=package://rtcosmik_ros/meshes/shoulder_mesh.STL scale=0.003600 0.003600 0.003600; visual mesh filename=package://rtcosmik_ros/meshes/upperarm_mesh.STL scale=0.005700 0.005500 0.006300
- link right_upperleg: mass 9.1 -> 6.15; geometry visual mesh filename=package://rtcosmik_ros/meshes/upperleg_mesh.STL scale=0.005600 0.005800 0.006300
Joints:
- joint joint_C7: origin xyz=-0.080403 0.304940 -0.001789 rpy=0.000000 -0.000000 0.000000 -> xyz=-0.078358 0.288973 -0.000239 rpy=0.000000 -0.000000 0.000000
- joint joint_Head: origin xyz=-0.042938 0.258525 -0.005349 rpy=0.000000 -0.000000 0.000000 -> xyz=-0.035738 0.259984 0.004340 rpy=0.000000 -0.000000 0.000000
- joint joint_L5MHD: origin xyz=0.138644 -0.035999 -0.041912 rpy=0.000000 -0.000000 0.000000 -> xyz=0.150688 -0.037942 -0.036893 rpy=0.000000 -0.000000 0.000000
- joint joint_LANK: origin xyz=-0.003708 -0.462206 -0.033679 rpy=0.000000 -0.000000 0.000000 -> xyz=-0.006134 -0.412509 -0.033854 rpy=0.000000 -0.000000 0.000000
- joint joint_LASI: origin xyz=0.084222 -0.002758 -0.115229 rpy=0.000000 -0.000000 0.000000 -> xyz=0.093734 -0.002485 -0.116798 rpy=0.000000 -0.000000 0.000000
- joint joint_LELB: origin xyz=0.013404 -0.278677 -0.018009 rpy=0.000000 -0.000000 0.000000 -> xyz=0.006774 -0.258750 -0.022203 rpy=0.000000 -0.000000 0.000000
- joint joint_LEar: origin xyz=-0.012661 0.127764 -0.077262 rpy=0.000000 -0.000000 0.000000 -> xyz=-0.009180 0.132749 -0.067623 rpy=0.000000 -0.000000 0.000000
- joint joint_LEye: origin xyz=0.075322 0.161414 -0.036531 rpy=0.000000 -0.000000 0.000000 -> xyz=0.071754 0.158247 -0.031755 rpy=0.000000 -0.000000 0.000000
- joint joint_LHEE: origin xyz=-0.054828 -0.033255 0.000761 rpy=0.000000 -0.000000 0.000000 -> xyz=-0.063737 -0.030079 0.002174 rpy=0.000000 -0.000000 0.000000
- joint joint_LKNE: origin xyz=0.009129 -0.395153 -0.046892 rpy=0.000000 -0.000000 0.000000 -> xyz=0.009525 -0.365019 -0.047785 rpy=0.000000 -0.000000 0.000000
- joint joint_LMANK: origin xyz=0.003952 -0.457384 0.031801 rpy=0.000000 -0.000000 0.000000 -> xyz=0.006049 -0.408895 0.031691 rpy=0.000000 -0.000000 0.000000
- joint joint_LMELB: origin xyz=-0.012587 -0.286336 0.056077 rpy=0.000000 -0.000000 0.000000 -> xyz=-0.006802 -0.272777 0.043744 rpy=0.000000 -0.000000 0.000000
- joint joint_LMID: origin xyz=-0.001265 -0.127797 -0.002368 rpy=0.000000 -0.000000 0.000000 -> xyz=-0.000050 -0.113695 -0.002826 rpy=0.000000 -0.000000 0.000000
- joint joint_LMKNE: origin xyz=-0.009133 -0.388279 0.063135 rpy=0.000000 -0.000000 0.000000 -> xyz=-0.008136 -0.362272 0.066465 rpy=0.000000 -0.000000 0.000000
- joint joint_LMWRI: origin xyz=-0.016401 -0.246420 0.009986 rpy=0.000000 -0.000000 0.000000 -> xyz=-0.012540 -0.236898 0.013217 rpy=0.000000 -0.000000 0.000000
- joint joint_LPIN: origin xyz=0.004875 -0.144521 0.024714 rpy=0.000000 -0.000000 0.000000 -> xyz=0.009820 -0.140516 0.028578 rpy=0.000000 -0.000000 0.000000
- joint joint_LPSI: origin xyz=-0.084374 0.002051 -0.058808 rpy=0.000000 -0.000000 0.000000 -> xyz=-0.095174 0.000664 -0.056749 rpy=0.000000 -0.000000 0.000000
- joint joint_LSHO: origin xyz=-0.011227 0.004744 -0.156694 rpy=0.000000 -0.000000 0.000000 -> xyz=-0.008268 0.002031 -0.142794 rpy=0.000000 -0.000000 0.000000
- joint joint_LTHU: origin xyz=0.017502 -0.101302 -0.042385 rpy=0.000000 -0.000000 0.000000 -> xyz=0.015813 -0.095688 -0.038832 rpy=0.000000 -0.000000 0.000000
- joint joint_LTOE: origin xyz=0.183317 -0.030757 0.027229 rpy=0.000000 -0.000000 0.000000 -> xyz=0.196040 -0.022068 0.024516 rpy=0.000000 -0.000000 0.000000
- joint joint_LWRI: origin xyz=-0.004162 -0.241738 -0.021819 rpy=0.000000 -0.000000 0.000000 -> xyz=-0.000848 -0.228065 -0.019986 rpy=0.000000 -0.000000 0.000000
- joint joint_Nose: origin xyz=0.117305 0.116548 -0.003687 rpy=0.000000 -0.000000 0.000000 -> xyz=0.109879 0.121166 -0.002977 rpy=0.000000 -0.000000 0.000000
- joint joint_R5MHD: origin xyz=0.131005 -0.052868 0.036635 rpy=0.000000 -0.000000 0.000000 -> xyz=0.136080 -0.054527 0.034125 rpy=0.000000 -0.000000 0.000000
- joint joint_RANK: origin xyz=-0.003593 -0.453700 0.030322 rpy=0.000000 -0.000000 0.000000 -> xyz=-0.003256 -0.405026 0.033622 rpy=0.000000 -0.000000 0.000000
- joint joint_RASI: origin xyz=0.084514 -0.003155 0.114142 rpy=0.000000 -0.000000 0.000000 -> xyz=0.091097 -0.002495 0.113532 rpy=0.000000 -0.000000 0.000000
- joint joint_RELB: origin xyz=0.012643 -0.274683 0.017820 rpy=0.000000 -0.000000 0.000000 -> xyz=0.010556 -0.249826 0.019504 rpy=0.000000 -0.000000 0.000000
- joint joint_REar: origin xyz=-0.010699 0.125607 0.066083 rpy=0.000000 -0.000000 0.000000 -> xyz=-0.009536 0.126169 0.071741 rpy=0.000000 -0.000000 0.000000
- joint joint_REye: origin xyz=0.076730 0.160508 0.026633 rpy=0.000000 -0.000000 0.000000 -> xyz=0.073543 0.155711 0.030654 rpy=0.000000 -0.000000 0.000000
- joint joint_RHEE: origin xyz=-0.053447 -0.046394 -0.008728 rpy=0.000000 -0.000000 0.000000 -> xyz=-0.062208 -0.045704 -0.007657 rpy=0.000000 -0.000000 0.000000
- joint joint_RKNE: origin xyz=0.011967 -0.399554 0.052019 rpy=0.000000 -0.000000 0.000000 -> xyz=0.008942 -0.367729 0.048517 rpy=0.000000 -0.000000 0.000000
- joint joint_RMANK: origin xyz=0.003366 -0.453382 -0.031911 rpy=0.000000 -0.000000 0.000000 -> xyz=0.002881 -0.406995 -0.031808 rpy=0.000000 -0.000000 0.000000
- joint joint_RMELB: origin xyz=-0.011456 -0.286480 -0.051546 rpy=0.000000 -0.000000 0.000000 -> xyz=-0.008915 -0.268327 -0.052669 rpy=0.000000 -0.000000 0.000000
- joint joint_RMID: origin xyz=-0.000233 -0.128281 0.000751 rpy=0.000000 -0.000000 0.000000 -> xyz=0.001444 -0.111730 0.002234 rpy=0.000000 -0.000000 0.000000
- joint joint_RMKNE: origin xyz=-0.010461 -0.398982 -0.057720 rpy=0.000000 -0.000000 0.000000 -> xyz=-0.007240 -0.366283 -0.063518 rpy=0.000000 -0.000000 0.000000
- joint joint_RMWRI: origin xyz=-0.013745 -0.245145 -0.011280 rpy=0.000000 -0.000000 0.000000 -> xyz=-0.013949 -0.239425 -0.009304 rpy=0.000000 -0.000000 0.000000
- joint joint_RPIN: origin xyz=-0.000626 -0.147241 -0.031849 rpy=0.000000 -0.000000 0.000000 -> xyz=0.004378 -0.141062 -0.035555 rpy=0.000000 -0.000000 0.000000
- joint joint_RPSI: origin xyz=-0.084832 -0.000319 0.055091 rpy=0.000000 -0.000000 0.000000 -> xyz=-0.092211 0.000311 0.056450 rpy=0.000000 -0.000000 0.000000
- joint joint_RSHO: origin xyz=-0.017031 -0.005065 0.152077 rpy=0.000000 -0.000000 0.000000 -> xyz=-0.009193 -0.005186 0.144428 rpy=0.000000 -0.000000 0.000000
- joint joint_RTHU: origin xyz=0.017843 -0.094398 0.044588 rpy=0.000000 -0.000000 0.000000 -> xyz=0.017719 -0.090181 0.032178 rpy=0.000000 -0.000000 0.000000
- joint joint_RTOE: origin xyz=0.175883 -0.039904 -0.033033 rpy=0.000000 -0.000000 0.000000 -> xyz=0.191634 -0.036677 -0.033431 rpy=0.000000 -0.000000 0.000000
- joint joint_RWRI: origin xyz=-0.004111 -0.242283 0.021845 rpy=0.000000 -0.000000 0.000000 -> xyz=-0.003602 -0.231802 0.019976 rpy=0.000000 -0.000000 0.000000
- joint joint_T11: origin xyz=-0.099289 0.206912 0.000960 rpy=0.000000 -0.000000 0.000000 -> xyz=-0.102714 0.186944 -0.006549 rpy=0.000000 -0.000000 0.000000
- joint joint_T6: origin xyz=-0.107234 0.176306 -0.003218 rpy=0.000000 -0.000000 0.000000 -> xyz=-0.105953 0.162893 -0.007823 rpy=0.000000 -0.000000 0.000000
- joint left_ankle_Z: origin xyz=0.000000 -0.459255 0.000000 rpy=0.000000 -0.000000 0.000000 -> xyz=0.000000 -0.410164 0.000000 rpy=0.000000 -0.000000 0.000000
- joint left_clavicle_joint_X: origin xyz=0.000000 0.287346 0.000000 rpy=0.000000 -0.000000 0.000000 -> xyz=0.000000 0.274077 0.000000 rpy=0.000000 -0.000000 0.000000
- joint left_elbow_Z: origin xyz=0.000000 -0.281772 0.000000 rpy=0.000000 -0.000000 0.000000 -> xyz=0.000000 -0.264839 0.000000 rpy=0.000000 -0.000000 0.000000
- joint left_hip_Z: origin xyz=0.015698 -0.085393 -0.082261 rpy=0.000000 -0.000000 0.000000 -> xyz=0.023965 -0.085296 -0.083085 rpy=0.000000 -0.000000 0.000000
- joint left_knee_Z: origin xyz=0.000000 -0.391086 0.000000 rpy=0.000000 -0.000000 0.000000 -> xyz=0.000000 -0.362862 0.000000 rpy=0.000000 -0.000000 0.000000
- joint left_shoulder_Z: origin xyz=0.004617 -0.048239 -0.154356 rpy=0.000000 -0.000000 0.000000 -> xyz=-0.001978 -0.045488 -0.143604 rpy=0.000000 -0.000000 0.000000
- joint left_wrist_Z: origin xyz=0.000000 -0.245200 0.000000 rpy=0.000000 -0.000000 0.000000 -> xyz=0.000000 -0.232336 0.000000 rpy=0.000000 -0.000000 0.000000
- joint middle_cervical_Z: origin xyz=0.000000 0.316179 0.000000 rpy=0.000000 -0.000000 0.000000 -> xyz=0.000000 0.294985 0.000000 rpy=0.000000 -0.000000 0.000000
- joint middle_thoracic_Z: origin xyz=0.000000 0.149427 0.000000 rpy=0.000000 -0.000000 0.000000 -> xyz=0.000000 0.135670 0.000000 rpy=0.000000 -0.000000 0.000000
- joint right_ankle_Z: origin xyz=0.000000 -0.452413 0.000000 rpy=0.000000 -0.000000 0.000000 -> xyz=0.000000 -0.405139 0.000000 rpy=0.000000 -0.000000 0.000000
- joint right_clavicle_joint_X: origin xyz=0.000000 0.287346 0.000000 rpy=0.000000 -0.000000 0.000000 -> xyz=0.000000 0.274077 0.000000 rpy=0.000000 -0.000000 0.000000
- joint right_elbow_Z: origin xyz=0.000000 -0.279813 0.000000 rpy=0.000000 -0.000000 0.000000 -> xyz=0.000000 -0.258374 0.000000 rpy=0.000000 -0.000000 0.000000
- joint right_hip_Z: origin xyz=0.015698 -0.084338 0.083342 rpy=0.000000 -0.000000 0.000000 -> xyz=0.023965 -0.085160 0.083224 rpy=0.000000 -0.000000 0.000000
- joint right_knee_Z: origin xyz=0.000000 -0.398015 0.000000 rpy=0.000000 -0.000000 0.000000 -> xyz=0.000000 -0.365901 0.000000 rpy=0.000000 -0.000000 0.000000
- joint right_shoulder_Z: origin xyz=-0.004617 -0.056811 0.154356 rpy=0.000000 -0.000000 0.000000 -> xyz=0.001978 -0.052199 0.143604 rpy=0.000000 -0.000000 0.000000
- joint right_wrist_Z: origin xyz=0.000000 -0.244295 0.000000 rpy=0.000000 -0.000000 0.000000 -> xyz=0.000000 -0.236234 0.000000 rpy=0.000000 -0.000000 0.000000
